File: interface/pcb/interface.sch (KiCad schematic (older format))
At the start: 0 parts

Commit message: PCB revisions
Changed lines of the file:
@@
 LIBS:SeeedOPL-Connector-2016
 LIBS:SeeedOPL-Inductor-2016
+LIBS:SeeedOPL-Display-2016
 LIBS:interface-cache
 EELAYER 25 0
@@
 $Descr A4 11693 8268
 encoding utf-8
-Sheet 1 8
+Sheet 1 7
 Title ""
 Date ""
@@
 $EndDescr
 $Sheet
-S 8800 2250 1500 750
+S 7700 2250 1500 750
 U 59C404DC
 F0 "SD Card" 59
 F1 "sdcard.sch" 59
-F2 "SD_SPI_CS" I L 8800 2600 59
-F3 "SD_SPI_MOSI" I L 8800 2900 59
-F4 "SD_SPI_SCK" I L 8800 2700 59
-F5 "SD_SPI_MISO" O L 8800 2800 59
-F6 "SD_CARD_DET_L" O L 8800 2400 59
+F2 "SD_SPI_CS" I L 7700 2600 59
+F3 "SD_SPI_MOSI" I L 7700 2900 59
+F4 "SD_SPI_SCK" I L 7700 2700 59
+F5 "SD_SPI_MISO" O L 7700 2800 59
+F6 "SD_CARD_DET_L" O L 7700 2400 59
 $EndSheet
 Wire Wire Line
-	8200 2400 8800 2400
+	7100 2400 7700 2400
 Wire Wire Line
-	8200 2600 8800 2600
+	7100 2600 7700 2600
 Wire Wire Line
-	8800 2700 8200 2700
+	7700 2700 7100 2700
 Wire Wire Line
-	8200 2800 8800 2800
+	7100 2800 7700 2800
 Wire Wire Line
-	8800 2900 8200 2900
+	7700 2900 7100 2900
 $Sheet
-S 6350 2250 1850 3200
-U 59C30A03
-F0 "STM32 MCU" 60
-F1 "mcu.sch" 60
-F2 "SD_CARD_DET" I R 8200 2400 59
-F3 "SD_SPI_CS" O R 8200 2600 59
-F4 "SD_SPI_SCK" O R 8200 2700 59
-F5 "SD_SPI_MISO" I R 8200 2800 59
-F6 "SD_SPI_MOSI" O R 8200 2900 59
-F7 "MDB_USART_VEND_TO_ST" I R 8200 5100 59
-F8 "MDB_USART_VEND_FROM_ST" O R 8200 5000 59
-F9 "TEMP_I2C_SCL" O R 8200 3400 59
-F10 "TEMP_I2C_SDA" B R 8200 3500 59
-F11 "CARD_BUZZ" O R 8200 4000 59
-F12 "CARD_LED" O R 8200 4100 59
-F13 "CARD_DATA0" O R 8200 4200 59
-F14 "CARD_DATA1" O R 8200 4300 59
-F15 "MDB_POWER_DET" I R 8200 4800 59
-F16 "LCD_DATA0" O L 6350 2400 59
-F17 "LCD_DATA1" O L 6350 2500 59
-F18 "LCD_DATA2" O L 6350 2600 59
-F19 "LCD_DATA3" O L 6350 2700 59
-F20 "LCD_RW" O L 6350 2850 59
-F21 "LCD_EN" O L 6350 2950 59
-F22 "LCD_RS" O L 6350 3050 59
-$EndSheet
-$Sheet
-S 8800 3300 1500 300
+S 7700 3300 1500 300
 U 59C737CF
 F0 "Temp Sensor" 59
 F1 "temp.sch" 59
-F2 "TEMP_ALARM" O R 10300 3400 59
-F3 "TEMP_I2C_SCL" I L 8800 3400 59
-F4 "TEMP_I2C_SDA" B L 8800 3500 59
+F2 "TEMP_ALARM" O R 9200 3400 59
+F3 "TEMP_I2C_SCL" I L 7700 3400 59
+F4 "TEMP_I2C_SDA" B L 7700 3500 59
 $EndSheet
 Wire Wire Line
-	8800 3500 8200 3500
+	7700 3500 7100 3500
 Wire Wire Line
-	8200 3400 8800 3400
+	7100 3400 7700 3400
 $Sheet
-S 8800 3900 1500 500
+S 7700 3900 1500 500
 U 59C747A0
 F0 "Wiegand RFID Reader" 59
 F1 "wiegand.sch" 59
-F2 "CARD_BUZZ" I L 8800 4000 59
-F3 "CARD_LED" I L 8800 4100 59
-F4 "CARD_WIEGAND_0" O L 8800 4200 59
-F5 "CARD_WIEGAND_1" O L 8800 4300 59
+F2 "CARD_BUZZ" I L 7700 4000 59
+F3 "CARD_LED" I L 7700 4100 59
+F4 "CARD_WIEGAND_0" O L 7700 4200 59
+F5 "CARD_WIEGAND_1" O L 7700 4300 59
 $EndSheet
 Wire Wire Line
-	8200 4300 8800 4300
+	7100 4300 7700 4300
 Wire Wire Line
-	8800 4300 8800 4200
+	7700 4300 7700 4200
 Wire Wire Line
-	8800 4200 8200 4200
+	7700 4200 7100 4200
 Wire Wire Line
-	8800 4100 8200 4100
+	7700 4100 7100 4100
 Wire Wire Line
-	8200 4000 8800 4000
+	7100 4000 7700 4000
 $Sheet
-S 8800 4700 1500 750
+S 7700 4700 1500 750
 U 59C7A00B
 F0 "MDB" 59
 F1 "mdb.sch" 59
-F2 "MDB_POWER_DET_L" O L 8800 4800 59
-F3 "MDB_TXO" I L 8800 5000 59
-F4 "MDB_RXI" O L 8800 5100 59
+F2 "MDB_POWER_DET_L" O L 7700 4800 59
+F3 "MDB_TXO" I L 7700 5000 59
+F4 "MDB_RXI" O L 7700 5100 59
 $EndSheet
 Wire Wire Line
-	8200 5000 8800 5000
+	7100 5000 7700 5000
 Wire Wire Line
-	8800 5100 8200 5100
+	7700 5100 7100 5100
 Wire Wire Line
-	8800 4800 8200 4800
-$Sheet
-S 4300 2250 1350 950
-U 59C8361F
-F0 "LCD" 59
-F1 "lcd.sch" 59
-F2 "LCD_RS" I R 5650 3050 59
-F3 "LCD_RW" I R 5650 2850 59
-F4 "LCD_EN" I R 5650 2950 59
-F5 "LCD_DATA0" I R 5650 2400 59
-F6 "LCD_DATA1" I R 5650 2500 59
-F7 "LCD_DATA2" I R 5650 2600 59
-F8 "LCD_DATA3" I R 5650 2700 59
-$EndSheet
-Wire Wire Line
-	5650 2400 6350 2400
-Wire Wire Line
-	6350 2500 5650 2500
-Wire Wire Line
-	5650 2600 6350 2600
-Wire Wire Line
-	6350 2700 5650 2700
-Wire Wire Line
-	5650 2850 6350 2850
-Wire Wire Line
-	6350 2950 5650 2950
-Wire Wire Line
-	5650 3050 6350 3050
+	7700 4800 7100 4800
 Text Notes 9100 7650 2    59   ~ 12
 24 September 2017
@@
 F1 "power.sch" 39
 $EndSheet
+$Sheet
+S 5250 2250 1850 3200
+U 59C30A03
+F0 "STM32 MCU" 60
+F1 "mcu.sch" 60
+F2 "SD_CARD_DET" I R 7100 2400 59
+F3 "SD_SPI_CS" O R 7100 2600 59
+F4 "SD_SPI_SCK" O R 7100 2700 59
+F5 "SD_SPI_MISO" I R 7100 2800 59
+F6 "SD_SPI_MOSI" O R 7100 2900 59
+F7 "MDB_USART_VEND_TO_ST" I R 7100 5100 59
+F8 "MDB_USART_VEND_FROM_ST" O R 7100 5000 59
+F9 "TEMP_I2C_SCL" O R 7100 3400 59
+F10 "TEMP_I2C_SDA" B R 7100 3500 59
+F11 "CARD_BUZZ" O R 7100 4000 59
+F12 "CARD_LED" O R 7100 4100 59
+F13 "CARD_DATA0" O R 7100 4200 59
+F14 "CARD_DATA1" O R 7100 4300 59
+F15 "MDB_POWER_DET" I R 7100 4800 59
+$EndSheet
 $EndSCHEMATC

Commit message: Partial BOM
Changed lines of the file:
@@
 EESchema Schematic File Version 2
+LIBS:interface-rescue
 LIBS:power
 LIBS:device
@@
 LIBS:tpd4s012
 LIBS:ap1509
-LIBS:device_big
 LIBS:SeeedOPL-Resistor-2016
 LIBS:SeeedOPL-Connector-2016
 LIBS:SeeedOPL-Inductor-2016
 LIBS:SeeedOPL-Display-2016
+LIBS:nhd-c0220biz
 LIBS:interface-cache
 EELAYER 25 0
@@
 $EndDescr
 $Sheet
-S 7700 2250 1500 750
+S 6200 2350 1500 750
 U 59C404DC
 F0 "SD Card" 59
 F1 "sdcard.sch" 59
-F2 "SD_SPI_CS" I L 7700 2600 59
-F3 "SD_SPI_MOSI" I L 7700 2900 59
-F4 "SD_SPI_SCK" I L 7700 2700 59
-F5 "SD_SPI_MISO" O L 7700 2800 59
-F6 "SD_CARD_DET_L" O L 7700 2400 59
+F2 "SD_SPI_CS" I L 6200 2700 59
+F3 "SD_SPI_MOSI" I L 6200 3000 59
+F4 "SD_SPI_SCK" I L 6200 2800 59
+F5 "SD_SPI_MISO" O L 6200 2900 59
+F6 "SD_CARD_DET_L" O L 6200 2500 59
 $EndSheet
 Wire Wire Line
-	7100 2400 7700 2400
+	5600 2500 6200 2500
 Wire Wire Line
-	7100 2600 7700 2600
+	5600 2700 6200 2700
 Wire Wire Line
-	7700 2700 7100 2700
+	6200 2800 5600 2800
 Wire Wire Line
-	7100 2800 7700 2800
+	5600 2900 6200 2900
 Wire Wire Line
-	7700 2900 7100 2900
+	6200 3000 5600 3000
 $Sheet
-S 7700 3300 1500 300
+S 6200 3400 1500 300
 U 59C737CF
 F0 "Temp Sensor" 59
 F1 "temp.sch" 59
-F2 "TEMP_ALARM" O R 9200 3400 59
-F3 "TEMP_I2C_SCL" I L 7700 3400 59
-F4 "TEMP_I2C_SDA" B L 7700 3500 59
+F2 "TEMP_ALARM" O R 7700 3500 59
+F3 "TEMP_I2C_SCL" I L 6200 3500 59
+F4 "TEMP_I2C_SDA" B L 6200 3600 59
 $EndSheet
 Wire Wire Line
-	7700 3500 7100 3500
+	6200 3600 5600 3600
 Wire Wire Line
-	7100 3400 7700 3400
+	5600 3500 6200 3500
 $Sheet
-S 7700 3900 1500 500
+S 6200 4000 1500 500
 U 59C747A0
 F0 "Wiegand RFID Reader" 59
 F1 "wiegand.sch" 59
-F2 "CARD_BUZZ" I L 7700 4000 59
-F3 "CARD_LED" I L 7700 4100 59
-F4 "CARD_WIEGAND_0" O L 7700 4200 59
-F5 "CARD_WIEGAND_1" O L 7700 4300 59
+F2 "CARD_BUZZ" I L 6200 4100 59
+F3 "CARD_LED" I L 6200 4200 59
+F4 "CARD_WIEGAND_0" O L 6200 4300 59
+F5 "CARD_WIEGAND_1" O L 6200 4400 59
 $EndSheet
 Wire Wire Line
-	7100 4300 7700 4300
+	5600 4400 6200 4400
 Wire Wire Line
-	7700 4300 7700 4200
+	6200 4400 6200 4300
 Wire Wire Line
-	7700 4200 7100 4200
+	6200 4300 5600 4300
 Wire Wire Line
-	7700 4100 7100 4100
+	6200 4200 5600 4200
 Wire Wire Line
-	7100 4000 7700 4000
+	5600 4100 6200 4100
 $Sheet
-S 7700 4700 1500 750
+S 6200 4800 1500 750
 U 59C7A00B
 F0 "MDB" 59
 F1 "mdb.sch" 59
-F2 "MDB_POWER_DET_L" O L 7700 4800 59
-F3 "MDB_TXO" I L 7700 5000 59
-F4 "MDB_RXI" O L 7700 5100 59
+F2 "MDB_POWER_DET_L" O L 6200 4900 59
+F3 "MDB_TXO" I L 6200 5100 59
+F4 "MDB_RXI" O L 6200 5200 59
 $EndSheet
 Wire Wire Line
-	7100 5000 7700 5000
+	5600 5100 6200 5100
 Wire Wire Line
-	7700 5100 7100 5100
+	6200 5200 5600 5200
 Wire Wire Line
-	7700 4800 7100 4800
+	6200 4900 5600 4900
 Text Notes 9100 7650 2    59   ~ 12
 24 September 2017
 $Sheet
-S 1250 2250 1800 950
+S 3750 1400 1150 650
 U 59C92DEF
 F0 "Power" 39
@@
 $EndSheet
 $Sheet
-S 5250 2250 1850 3200
+S 3750 2350 1850 3200
 U 59C30A03
 F0 "STM32 MCU" 60
 F1 "mcu.sch" 60
-F2 "SD_CARD_DET" I R 7100 2400 59
-F3 "SD_SPI_CS" O R 7100 2600 59
-F4 "SD_SPI_SCK" O R 7100 2700 59
-F5 "SD_SPI_MISO" I R 7100 2800 59
-F6 "SD_SPI_MOSI" O R 7100 2900 59
-F7 "MDB_USART_VEND_TO_ST" I R 7100 5100 59
-F8 "MDB_USART_VEND_FROM_ST" O R 7100 5000 59
-F9 "TEMP_I2C_SCL" O R 7100 3400 59
-F10 "TEMP_I2C_SDA" B R 7100 3500 59
-F11 "CARD_BUZZ" O R 7100 4000 59
-F12 "CARD_LED" O R 7100 4100 59
-F13 "CARD_DATA0" O R 7100 4200 59
-F14 "CARD_DATA1" O R 7100 4300 59
-F15 "MDB_POWER_DET" I R 7100 4800 59
+F2 "SD_CARD_DET" I R 5600 2500 59
+F3 "SD_SPI_CS" O R 5600 2700 59
+F4 "SD_SPI_SCK" O R 5600 2800 59
+F5 "SD_SPI_MISO" I R 5600 2900 59
+F6 "SD_SPI_MOSI" O R 5600 3000 59
+F7 "MDB_USART_VEND_TO_ST" I R 5600 5200 59
+F8 "MDB_USART_VEND_FROM_ST" O R 5600 5100 59
+F9 "TEMP_I2C_SCL" O R 5600 3500 59
+F10 "TEMP_I2C_SDA" B R 5600 3600 59
+F11 "CARD_BUZZ" O R 5600 4100 59
+F12 "CARD_LED" O R 5600 4200 59
+F13 "CARD_DATA0" O R 5600 4300 59
+F14 "CARD_DATA1" O R 5600 4400 59
+F15 "MDB_POWER_DET" I R 5600 4900 59
 $EndSheet
 $EndSCHEMATC

Commit message: Start of layout
Changed lines of the file:
@@
 F7 "MDB_USART_VEND_TO_ST" I R 5600 5200 59
 F8 "MDB_USART_VEND_FROM_ST" O R 5600 5100 59
-F9 "TEMP_I2C_SCL" O R 5600 3500 59
-F10 "TEMP_I2C_SDA" B R 5600 3600 59
-F11 "CARD_BUZZ" O R 5600 4100 59
-F12 "CARD_LED" O R 5600 4200 59
-F13 "CARD_DATA0" O R 5600 4300 59
-F14 "CARD_DATA1" O R 5600 4400 59
-F15 "MDB_POWER_DET" I R 5600 4900 59
+F9 "CARD_BUZZ" O R 5600 4100 59
+F10 "CARD_LED" O R 5600 4200 59
+F11 "CARD_DATA0" O R 5600 4300 59
+F12 "CARD_DATA1" O R 5600 4400 59
+F13 "MDB_POWER_DET" I R 5600 4900 59
+F14 "I2C_SCL" O R 5600 3500 60
+F15 "I2C_SDA" B R 5600 3600 60
 $EndSheet
 $EndSCHEMATC
