File: interface/pcb/mcu.sch (KiCad schematic (older format))
At the start: 37 parts, among them P1 SWD_DEBUG, P2 EXTRA_GPIO, Q2 BSS84, SW1 RESET_BTN, SW2 BUTTON1, SW3 BUTTON2, U1 STM32F103CBTx, U2 TPD4S012, X1 12Mhz

Commit message: PCB revisions
Parts:
- removed R10: 10K, symbol R
- removed R11: 100K, symbol R
Connections:
- net labels added: I2C_SCL, I2C_SDA
- net labels removed: LCD_DATA0, LCD_DATA1, LCD_DATA2, LCD_DATA3, LCD_EN, LCD_RS, LCD_RW, TEMP_I2C_SCL, TEMP_I2C_SDA
- wire segments 152 -> 165
Other:
- note added: "NO-STUFF Q2\nNO-STUFF R21"
Changed lines of the file:
@@
 LIBS:SeeedOPL-Connector-2016
 LIBS:SeeedOPL-Inductor-2016
+LIBS:SeeedOPL-Display-2016
 LIBS:interface-cache
 EELAYER 25 0
@@
 $Descr A3 16535 11693
 encoding utf-8
-Sheet 3 8
+Sheet 7 7
 Title ""
 Date ""
@@
 	0    -1   -1   0
 $EndComp
-$Comp
-L R R10
-U 1 1 59C38977
-P 3850 8800
-F 0 "R10" V 3930 8800 50  0000 C CNN
-F 1 "10K" V 3850 8800 50  0000 C CNN
-F 2 "" V 3780 8800 50  0001 C CNN
-F 3 "" H 3850 8800 50  0000 C CNN
-	1    3850 8800
-	-1   0    0    1
-$EndComp
-$Comp
-L +3.3V #PWR031
-U 1 1 59C389F6
-P 3850 8650
-F 0 "#PWR031" H 3850 8500 50  0001 C CNN
-F 1 "+3.3V" H 3850 8790 50  0000 C CNN
-F 2 "" H 3850 8650 50  0000 C CNN
-F 3 "" H 3850 8650 50  0000 C CNN
-	1    3850 8650
-	1    0    0    -1
-$EndComp
-$Comp
-L R R11
-U 1 1 59C38A40
-P 3850 9500
-F 0 "R11" V 3930 9500 50  0000 C CNN
-F 1 "100K" V 3850 9500 50  0000 C CNN
-F 2 "" V 3780 9500 50  0001 C CNN
-F 3 "" H 3850 9500 50  0000 C CNN
-	1    3850 9500
-	-1   0    0    1
-$EndComp
-$Comp
-L GND #PWR032
-U 1 1 59C38BE5
-P 3850 9700
-F 0 "#PWR032" H 3850 9450 50  0001 C CNN
-F 1 "GND" H 3850 9550 50  0000 C CNN
-F 2 "" H 3850 9700 50  0000 C CNN
-F 3 "" H 3850 9700 50  0000 C CNN
-	1    3850 9700
-	1    0    0    -1
-$EndComp
-Wire Wire Line
-	7900 2550 7900 3350
+Wire Wire Line
+	7900 2550 7900 2800
+Wire Wire Line
+	7900 2800 7900 3350
 Wire Wire Line
 	8000 3350 8000 2800
 Wire Wire Line
-	7900 2800 8100 2800
+	7900 2800 8000 2800
+Wire Wire Line
+	8000 2800 8100 2800
 Connection ~ 7900 2800
 Wire Wire Line
@@
 	8100 7250 8100 6950
 Wire Wire Line
-	7900 7250 8100 7250
-Wire Wire Line
-	7900 6950 7900 7800
+	7900 7250 8000 7250
+Wire Wire Line
+	8000 7250 8100 7250
+Wire Wire Line
+	7900 6950 7900 7250
+Wire Wire Line
+	7900 7250 7900 7800
 Wire Wire Line
 	8000 6950 8000 7250
@@
 Connection ~ 7900 7250
 Wire Wire Line
-	8200 6950 8200 7350
+	8200 6950 8200 7250
+Wire Wire Line
+	8200 7250 8200 7350
 Wire Wire Line
 	8200 7650 8200 7800
@@
 	4900 3750 5200 3750
 Wire Wire Line
-	4900 2700 4900 3750
-Wire Wire Line
-	4900 2800 5900 2800
+	4900 2700 4900 2800
+Wire Wire Line
+	4900 2800 4900 3750
+Wire Wire Line
+	4900 2800 5600 2800
+Wire Wire Line
+	5600 2800 5900 2800
 Connection ~ 4900 2800
 Wire Wire Line
@@
 	2100 4150 5200 4150
 Wire Wire Line
-	2100 3550 2100 4150
+	2100 3550 2100 3700
+Wire Wire Line
+	2100 3700 2100 4150
 Wire Wire Line
 	1650 3750 1650 3700
@@
 Connection ~ 2100 3700
 Wire Wire Line
-	2100 4350 5200 4350
+	2100 4350 2500 4350
+Wire Wire Line
+	2500 4350 5200 4350
 Wire Wire Line
 	5200 4450 2750 4450
@@
 	2750 4450 2750 4750
 Wire Wire Line
-	2750 4750 2100 4750
+	2750 4750 2500 4750
+Wire Wire Line
+	2500 4750 2100 4750
 Connection ~ 2500 4750
 Connection ~ 2500 4350
@@
 	1800 4350 1650 4350
 Wire Wire Line
-	1650 4350 1650 4850
+	1650 4350 1650 4750
+Wire Wire Line
+	1650 4750 1650 4850
 Wire Wire Line
 	1650 4750 1800 4750
@@
 	1900 9100 1900 8650
 Wire Wire Line
-	2750 9100 3850 9100
-Wire Wire Line
-	2750 9200 3850 9200
+	2750 9100 3600 9100
+Wire Wire Line
+	2750 9200 3600 9200
 Wire Wire Line
 	2750 9500 3600 9500
@@
 	2250 9200 1900 9200
 Wire Wire Line
-	1900 9200 1900 9700
+	1900 9200 1900 9300
+Wire Wire Line
+	1900 9300 1900 9700
 Wire Wire Line
 	2250 9300 1900 9300
@@
 	4300 5350 3900 5350
 Wire Wire Line
-	3850 9100 3850 8950
-Wire Wire Line
-	3850 9200 3850 9350
-Wire Wire Line
-	3850 9650 3850 9700
-Wire Wire Line
 	11000 6450 11150 6450
 Wire Wire Line
 	11000 6350 11250 6350
 Wire Wire Line
-	2250 5850 5200 5850
-Wire Wire Line
-	2250 5950 5200 5950
+	2250 5850 2550 5850
+Wire Wire Line
+	2550 5850 5200 5850
+Wire Wire Line
+	2250 5950 2800 5950
+Wire Wire Line
+	2800 5950 5200 5950
 Text Notes 2500 10250 0    98   ~ 20
 Debugging
@@
 	13300 8250 13950 8250
 Wire Wire Line
-	13300 6850 13300 8250
-Wire Wire Line
-	13450 7050 13450 8150
+	13300 6850 13300 7150
+Wire Wire Line
+	13300 7150 13300 7950
+Wire Wire Line
+	13300 7950 13300 8250
+Wire Wire Line
+	13450 7050 13450 8050
+Wire Wire Line
+	13450 8050 13450 8150
 Wire Wire Line
 	13450 8150 13950 8150
@@
 	11000 5950 15150 5950
 Wire Wire Line
-	15150 5850 15150 6050
+	15150 5850 15150 5950
+Wire Wire Line
+	15150 5950 15150 6050
 Connection ~ 15150 5950
 $Comp
@@
 $EndComp
 Text HLabel 2250 5850 0    59   Output ~ 0
-TEMP_I2C_SCL
+I2C_SCL
 Text HLabel 2250 5950 0    59   BiDi ~ 0
-TEMP_I2C_SDA
+I2C_SDA
 Wire Wire Line
 	2550 5700 2550 5850
@@
 MDB_POWER_DET
 Wire Wire Line
-	11000 5550 12000 5550
-Wire Wire Line
-	12000 5650 11000 5650
-Wire Wire Line
-	11000 5750 12000 5750
-Wire Wire Line
-	12000 5850 11000 5850
-Text HLabel 12000 5550 2    59   Output ~ 0
-LCD_DATA0
-Text HLabel 12000 5650 2    59   Output ~ 0
-LCD_DATA1
-Text HLabel 12000 5750 2    59   Output ~ 0
-LCD_DATA2
-Text HLabel 12000 5850 2    59   Output ~ 0
-LCD_DATA3
-Wire Wire Line
 	3900 5050 5200 5050
-Wire Wire Line
-	11000 5450 12000 5450
-Wire Wire Line
-	11000 5150 12000 5150
-Wire Wire Line
-	12000 5050 11000 5050
-Text HLabel 12000 5050 2    59   Output ~ 0
-LCD_RW
-Text HLabel 12000 5150 2    59   Output ~ 0
-LCD_EN
-Text HLabel 12000 5450 2    59   Output ~ 0
-LCD_RS
 Wire Wire Line
 	5200 4650 3900 4650
@@
 	7200 9600 7350 9600
 Wire Wire Line
-	7350 9150 7350 9700
+	7350 9150 7350 9600
+Wire Wire Line
+	7350 9600 7350 9700
 Wire Wire Line
 	7200 9150 7350 9150
 Connection ~ 7350 9600
 Wire Wire Line
-	5250 9600 6600 9600
-Wire Wire Line
-	5250 9150 6600 9150
+	5250 9600 6150 9600
+Wire Wire Line
+	6150 9600 6600 9600
+Wire Wire Line
+	5250 9150 5950 9150
+Wire Wire Line
+	5950 9150 6600 9150
 Wire Wire Line
 	5950 9150 5950 8950
@@
 	9200 9050 9400 9050
 Wire Wire Line
-	9200 8650 9200 9050
+	9200 8650 9200 8800
+Wire Wire Line
+	9200 8800 9200 9050
 $Comp
 L +3.3V #PWR042
@@
 $EndComp
 Wire Wire Line
-	14450 8600 14450 8700
+	14450 8600 14450 8650
+Wire Wire Line
+	14450 8650 14450 8700
 Wire Wire Line
 	14450 7800 14450 7700
@@
 Text Notes 14800 8850 0    59   ~ 0
 320010018
+Text Notes 14400 7050 0    60   ~ 0
+NO-STUFF Q2\nNO-STUFF R21
 $EndSCHEMATC

Commit message: Partial BOM
Parts:
- added C19, C20: 1uF, Capacitors_SMD:C_0402, symbol C
- added C24: 0.1uF, Capacitors_SMD:C_0402, symbol C
- added LCD1: NHD-C0220BiZ, symbol NHD-C0220BiZ
- added R10, R11, R43: 10K, symbol R
- added R44: 20, symbol R
- SW1, SW2, SW3: footprint (none) -> Buttons_Switches_THT:SW_PUSH_6mm
- U1: footprint LQFP48 -> Housings_QFP:LQFP-48_7x7mm_Pitch0.5mm
Connections:
- net labels added: I2C_LCD_SCL, I2C_LCD_SDA, LCD_RESET, PA8
- net labels removed: PB2
- wire segments 165 -> 177
- no-connect marks 5 -> 9
Other:
- moved on the sheet: C10, C7, C8, C9, R12, R7, R8

Commit message: Start of layout
Parts:
- JP1: footprint (none) -> SeeedOPL-Connector-2016:USB4+2-2.5-90D-15.8X12MM
- LCD1: footprint (none) -> NHD-C0220BiZ:NHD-C0220BiZ
- P1: footprint (none) -> Pin_Headers:Pin_Header_Straight_2x05
- P2: footprint (none) -> Sockets_MOLEX_KK-System:Socket_MOLEX-KK-RM2-54mm_Lock_6pin_straight
- Q2: footprint (none) -> TO_SOT_Packages_SMD:SOT-23
- R10, R11, R12, R13, R14, R15, R16, R17, R18, R19, R20, R21, R22, R23, R43, R44, R7, R8, R9: footprint (none) -> Resistors_SMD:R_0402
- SW1, SW2, SW3: footprint Buttons_Switches_THT:SW_PUSH_6mm -> Buttons_Switches_ThroughHole:SW_PUSH_SMALL
- U2: footprint (none) -> Housings_SON:Fairchild_MicroPak-6_1.0x1.45mm_P0.5mm
- X1: footprint (none) -> SeeedOPL-Crystal Oscillator-2016:X2-SMD-5.0X3.2X1.3MM
