File: interface/pcb/mdb.sch (KiCad schematic (older format))
At the start: 25 parts, among them P5 MDB, Q7 MMBF170, Q8 MMBF170, U4 74HC14, U5 4N29, U6 4N29, U7 6N137

Commit message: PCB revisions
Parts:
- added JP?: Jumper_NO_Small, symbol Jumper_NO_Small
Connections:
- net GND: now also JP?.2
- net MDB_POWER_DET_L: now also JP?.1
Other:
- note added: "Closing JP disables \ndetector."
- moved on the sheet: D4, D5, Q7, Q8, R35, R36
Changed lines of the file:
@@
 LIBS:SeeedOPL-Connector-2016
 LIBS:SeeedOPL-Inductor-2016
+LIBS:SeeedOPL-Display-2016
 LIBS:interface-cache
 EELAYER 25 0
@@
 $Descr A4 11693 8268
 encoding utf-8
-Sheet 6 8
+Sheet 5 7
 Title ""
 Date ""
@@
 RX
 Wire Wire Line
-	2300 6550 2800 6550
-Text Label 2300 6550 0    59   ~ 0
+	1250 6500 1750 6500
+Text Label 1250 6500 0    59   ~ 0
 TX_DRIVE
 $Comp
 L GND #PWR074
 U 1 1 59C94C59
-P 3100 6850
-F 0 "#PWR074" H 3100 6600 50  0001 C CNN
-F 1 "GND" H 3100 6700 50  0000 C CNN
-F 2 "" H 3100 6850 50  0000 C CNN
-F 3 "" H 3100 6850 50  0000 C CNN
-	1    3100 6850
-	1    0    0    -1
-$EndComp
-Wire Wire Line
-	3100 6700 3100 6850
-Wire Wire Line
-	3100 6300 3100 6250
+P 2050 6800
+F 0 "#PWR074" H 2050 6550 50  0001 C CNN
+F 1 "GND" H 2050 6650 50  0000 C CNN
+F 2 "" H 2050 6800 50  0000 C CNN
+F 3 "" H 2050 6800 50  0000 C CNN
+	1    2050 6800
+	1    0    0    -1
+$EndComp
+Wire Wire Line
+	2050 6650 2050 6800
+Wire Wire Line
+	2050 6250 2050 6200
 $Comp
 L LED D4
 U 1 1 59C94C61
-P 3100 6050
-F 0 "D4" H 3100 6150 50  0000 C CNN
-F 1 "MDB_TX" H 3100 5950 50  0000 C CNN
-F 2 "LEDs:LED_0603" H 3100 6050 50  0001 C CNN
-F 3 "" H 3100 6050 50  0000 C CNN
-	1    3100 6050
+P 2050 6000
+F 0 "D4" H 2050 6100 50  0000 C CNN
+F 1 "MDB_TX" H 2050 5900 50  0000 C CNN
+F 2 "LEDs:LED_0603" H 2050 6000 50  0001 C CNN
+F 3 "" H 2050 6000 50  0000 C CNN
+	1    2050 6000
 	0    -1   -1   0
 $EndComp
@@
 L R R35
 U 1 1 59C94C68
-P 3100 5700
-F 0 "R35" V 3180 5700 50  0000 C CNN
-F 1 "330" V 3100 5700 50  0000 C CNN
-F 2 "" V 3030 5700 50  0001 C CNN
-F 3 "" H 3100 5700 50  0000 C CNN
-	1    3100 5700
+P 2050 5650
+F 0 "R35" V 2130 5650 50  0000 C CNN
+F 1 "330" V 2050 5650 50  0000 C CNN
+F 2 "" V 1980 5650 50  0001 C CNN
+F 3 "" H 2050 5650 50  0000 C CNN
+	1    2050 5650
 	-1   0    0    1
 $EndComp
@@
 L +3.3V #PWR075
 U 1 1 59C94C6F
-P 3100 5550
-F 0 "#PWR075" H 3100 5400 50  0001 C CNN
-F 1 "+3.3V" H 3100 5690 50  0000 C CNN
-F 2 "" H 3100 5550 50  0000 C CNN
-F 3 "" H 3100 5550 50  0000 C CNN
-	1    3100 5550
+P 2050 5500
+F 0 "#PWR075" H 2050 5350 50  0001 C CNN
+F 1 "+3.3V" H 2050 5640 50  0000 C CNN
+F 2 "" H 2050 5500 50  0000 C CNN
+F 3 "" H 2050 5500 50  0000 C CNN
+	1    2050 5500
 	1    0    0    -1
 $EndComp
@@
 L MMBF170 Q7
 U 1 1 59C94C75
-P 3000 6500
-F 0 "Q7" H 3200 6575 50  0000 L CNN
-F 1 "MMBF170" H 3200 6500 50  0000 L CNN
-F 2 "TO_SOT_Packages_SMD:SOT-23" H 3200 6425 50  0000 L CIN
-F 3 "" H 3000 6500 50  0000 L CNN
-	1    3000 6500
-	1    0    0    -1
-$EndComp
-Wire Wire Line
-	3800 6550 4300 6550
-Text Label 3800 6550 0    59   ~ 0
+P 1950 6450
+F 0 "Q7" H 2150 6525 50  0000 L CNN
+F 1 "MMBF170" H 2150 6450 50  0000 L CNN
+F 2 "TO_SOT_Packages_SMD:SOT-23" H 2150 6375 50  0000 L CIN
+F 3 "" H 1950 6450 50  0000 L CNN
+	1    1950 6450
+	1    0    0    -1
+$EndComp
+Wire Wire Line
+	3500 6500 4000 6500
+Text Label 3500 6500 0    59   ~ 0
 RX
 $Comp
 L GND #PWR076
 U 1 1 59C94D95
-P 4600 6850
-F 0 "#PWR076" H 4600 6600 50  0001 C CNN
-F 1 "GND" H 4600 6700 50  0000 C CNN
-F 2 "" H 4600 6850 50  0000 C CNN
-F 3 "" H 4600 6850 50  0000 C CNN
-	1    4600 6850
-	1    0    0    -1
-$EndComp
-Wire Wire Line
-	4600 6700 4600 6850
-Wire Wire Line
-	4600 6300 4600 6250
+P 4300 6800
+F 0 "#PWR076" H 4300 6550 50  0001 C CNN
+F 1 "GND" H 4300 6650 50  0000 C CNN
+F 2 "" H 4300 6800 50  0000 C CNN
+F 3 "" H 4300 6800 50  0000 C CNN
+	1    4300 6800
+	1    0    0    -1
+$EndComp
+Wire Wire Line
+	4300 6650 4300 6800
+Wire Wire Line
+	4300 6250 4300 6200
 $Comp
 L LED D5
 U 1 1 59C94D9D
-P 4600 6050
-F 0 "D5" H 4600 6150 50  0000 C CNN
-F 1 "MDB_RX" H 4600 5950 50  0000 C CNN
-F 2 "LEDs:LED_0603" H 4600 6050 50  0001 C CNN
-F 3 "" H 4600 6050 50  0000 C CNN
-	1    4600 6050
+P 4300 6000
+F 0 "D5" H 4300 6100 50  0000 C CNN
+F 1 "MDB_RX" H 4300 5900 50  0000 C CNN
+F 2 "LEDs:LED_0603" H 4300 6000 50  0001 C CNN
+F 3 "" H 4300 6000 50  0000 C CNN
+	1    4300 6000
 	0    -1   -1   0
 $EndComp
@@
 L R R36
 U 1 1 59C94DA4
-P 4600 5700
-F 0 "R36" V 4680 5700 50  0000 C CNN
-F 1 "330" V 4600 5700 50  0000 C CNN
-F 2 "" V 4530 5700 50  0001 C CNN
-F 3 "" H 4600 5700 50  0000 C CNN
-	1    4600 5700
+P 4300 5650
+F 0 "R36" V 4380 5650 50  0000 C CNN
+F 1 "330" V 4300 5650 50  0000 C CNN
+F 2 "" V 4230 5650 50  0001 C CNN
+F 3 "" H 4300 5650 50  0000 C CNN
+	1    4300 5650
 	-1   0    0    1
 $EndComp
@@
 L +3.3V #PWR077
 U 1 1 59C94DAB
-P 4600 5550
-F 0 "#PWR077" H 4600 5400 50  0001 C CNN
-F 1 "+3.3V" H 4600 5690 50  0000 C CNN
-F 2 "" H 4600 5550 50  0000 C CNN
-F 3 "" H 4600 5550 50  0000 C CNN
-	1    4600 5550
+P 4300 5500
+F 0 "#PWR077" H 4300 5350 50  0001 C CNN
+F 1 "+3.3V" H 4300 5640 50  0000 C CNN
+F 2 "" H 4300 5500 50  0000 C CNN
+F 3 "" H 4300 5500 50  0000 C CNN
+	1    4300 5500
 	1    0    0    -1
 $EndComp
@@
 L MMBF170 Q8
 U 1 1 59C94DB1
-P 4500 6500
-F 0 "Q8" H 4700 6575 50  0000 L CNN
-F 1 "MMBF170" H 4700 6500 50  0000 L CNN
-F 2 "TO_SOT_Packages_SMD:SOT-23" H 4700 6425 50  0000 L CIN
-F 3 "" H 4500 6500 50  0000 L CNN
-	1    4500 6500
-	1    0    0    -1
-$EndComp
-Text Notes 3300 7250 0    79   ~ 16
+P 4200 6450
+F 0 "Q8" H 4400 6525 50  0000 L CNN
+F 1 "MMBF170" H 4400 6450 50  0000 L CNN
+F 2 "TO_SOT_Packages_SMD:SOT-23" H 4400 6375 50  0000 L CIN
+F 3 "" H 4200 6450 50  0000 L CNN
+	1    4200 6450
+	1    0    0    -1
+$EndComp
+Text Notes 2800 7200 0    79   ~ 16
 MDB Activity LEDs
 $Comp
@@
 NoConn ~ 6250 2150
 NoConn ~ 6250 3950
+$Comp
+L Jumper_NO_Small JP?
+U 1 1 5A273710
+P 5850 2450
+F 0 "JP?" H 5850 2530 50  0000 C CNN
+F 1 "Jumper_NO_Small" H 5860 2390 50  0001 C CNN
+F 2 "" H 5850 2450 50  0000 C CNN
+F 3 "" H 5850 2450 50  0000 C CNN
+	1    5850 2450
+	1    0    0    -1
+$EndComp
+Wire Wire Line
+	5750 2450 5650 2450
+Wire Wire Line
+	5650 2450 5650 2250
+Connection ~ 5650 2250
+Wire Wire Line
+	5950 2450 6050 2450
+Connection ~ 6050 2450
+Text Notes 5200 2100 0    60   ~ 0
+Closing JP disables \ndetector.
 $EndSCHEMATC

Commit message: Partial BOM
Parts:
- D4, D5: symbol LED -> LED-RESCUE-interface
- P5: footprint (none) -> Sockets_MOLEX_KK-System:Socket_MOLEX-KK-RM2-54mm_Lock_5pin_straight
- Q7, Q8: footprint TO_SOT_Packages_SMD:SOT-23 -> TO_SOT_Packages_SMD:SOT-323_SC-70
- R35, R36, R37, R38, R39, R40, R41, R42: footprint (none) -> Resistors_SMD:R_0402
- U4: footprint (none) -> Housings_SOIC:SOIC-14_3.9x8.7mm_Pitch1.27mm
- U5, U6: footprint DIP-6 -> Housings_DIP:DIP-6_W7.62mm_Socket
- U7: footprint DIP-8 -> Housings_DIP:DIP-8_W7.62mm_Socket
- W12, W13, W14, W15, W16: footprint (none) -> Measurement_Points:Test_Point
- gave numbers to parts that had none: 1
Changed lines of the file:
@@
 EESchema Schematic File Version 2
+LIBS:interface-rescue
 LIBS:power
 LIBS:device
@@
 LIBS:tpd4s012
 LIBS:ap1509
-LIBS:device_big
 LIBS:SeeedOPL-Resistor-2016
 LIBS:SeeedOPL-Connector-2016
 LIBS:SeeedOPL-Inductor-2016
 LIBS:SeeedOPL-Display-2016
+LIBS:nhd-c0220biz
 LIBS:interface-cache
 EELAYER 25 0
@@
 F 0 "U6" H 6350 3350 50  0000 L CNN
 F 1 "4N29" H 6550 3350 50  0000 L CNN
-F 2 "DIP-6" H 6350 2950 50  0000 L CIN
+F 2 "Housings_DIP:DIP-6_W7.62mm_Socket" H 6350 2950 50  0000 L CIN
 F 3 "" H 6550 3150 50  0000 L CNN
 	1    6550 3150
@@
 F 0 "U5" H 6350 2450 50  0000 L CNN
 F 1 "4N29" H 6550 2450 50  0000 L CNN
-F 2 "DIP-6" H 6350 2050 50  0000 L CIN
+F 2 "Housings_DIP:DIP-6_W7.62mm_Socket" H 6350 2050 50  0000 L CIN
 F 3 "" H 6550 2250 50  0000 L CNN
 	1    6550 2250
@@
 F 0 "U7" H 6350 4350 50  0000 L CNN
 F 1 "6N137" H 6550 4350 50  0000 L CNN
-F 2 "DIP-8" H 6350 3750 50  0000 L CIN
+F 2 "Housings_DIP:DIP-8_W7.62mm_Socket" H 6350 3750 50  0000 L CIN
 F 3 "" H 6550 4050 50  0000 L CNN
 	1    6550 4050
@@
 F 0 "P5" H 9450 2650 50  0000 C CNN
 F 1 "MDB" V 9550 2350 50  0000 C CNN
-F 2 "" H 9450 2350 50  0001 C CNN
+F 2 "Sockets_MOLEX_KK-System:Socket_MOLEX-KK-RM2-54mm_Lock_5pin_straight" H 9450 2350 50  0001 C CNN
 F 3 "" H 9450 2350 50  0000 C CNN
 	1    9450 2350
@@
 F 0 "R41" V 7780 2150 50  0000 C CNN
 F 1 "100" V 7700 2150 50  0000 C CNN
-F 2 "" V 7630 2150 50  0001 C CNN
+F 2 "Resistors_SMD:R_0402" V 7630 2150 50  0001 C CNN
 F 3 "" H 7700 2150 50  0000 C CNN
 	1    7700 2150
@@
 F 0 "R42" V 7780 3950 50  0000 C CNN
 F 1 "1K" V 7700 3950 50  0000 C CNN
-F 2 "" V 7630 3950 50  0001 C CNN
+F 2 "Resistors_SMD:R_0402" V 7630 3950 50  0001 C CNN
 F 3 "" H 7700 3950 50  0000 C CNN
 	1    7700 3950
@@
 F 0 "R37" V 4930 1800 50  0000 C CNN
 F 1 "10K" V 4850 1800 50  0000 C CNN
-F 2 "" V 4780 1800 50  0001 C CNN
+F 2 "Resistors_SMD:R_0402" V 4780 1800 50  0001 C CNN
 F 3 "" H 4850 1800 50  0000 C CNN
 	1    4850 1800
@@
 $EndComp
 $Comp
-L +3.3V #PWR067
+L +3.3V #PWR030
 U 1 1 59C7A9C9
 P 4850 1550
-F 0 "#PWR067" H 4850 1400 50  0001 C CNN
+F 0 "#PWR030" H 4850 1400 50  0001 C CNN
 F 1 "+3.3V" H 4850 1690 50  0000 C CNN
 F 2 "" H 4850 1550 50  0000 C CNN
@@
 LOW when the vending \nmachine is powered.
 $Comp
-L GND #PWR068
+L GND #PWR031
 U 1 1 59C7AA95
 P 6050 4400
-F 0 "#PWR068" H 6050 4150 50  0001 C CNN
+F 0 "#PWR031" H 6050 4150 50  0001 C CNN
 F 1 "GND" H 6050 4250 50  0000 C CNN
 F 2 "" H 6050 4400 50  0000 C CNN
@@
 F 0 "U4" H 4650 3150 50  0000 C CNN
 F 1 "74HC14" H 4700 2950 50  0000 C CNN
-F 2 "" H 4500 3050 50  0001 C CNN
+F 2 "Housings_SOIC:SOIC-14_3.9x8.7mm_Pitch1.27mm" H 4500 3050 50  0001 C CNN
 F 3 "" H 4500 3050 50  0000 C CNN
 	1    4500 3050
@@
 F 0 "R39" V 5780 3050 50  0000 C CNN
 F 1 "1K" V 5700 3050 50  0000 C CNN
-F 2 "" V 5630 3050 50  0001 C CNN
+F 2 "Resistors_SMD:R_0402" V 5630 3050 50  0001 C CNN
 F 3 "" H 5700 3050 50  0000 C CNN
 	1    5700 3050
@@
 F 0 "U4" H 4650 4250 50  0000 C CNN
 F 1 "74HC14" H 4700 4050 50  0000 C CNN
-F 2 "" H 4500 4150 50  0001 C CNN
+F 2 "Housings_SOIC:SOIC-14_3.9x8.7mm_Pitch1.27mm" H 4500 4150 50  0001 C CNN
 F 3 "" H 4500 4150 50  0000 C CNN
 	2    4500 4150
@@
 F 0 "U4" H 4650 4750 50  0000 C CNN
 F 1 "74HC14" H 4700 4550 50  0000 C CNN
-F 2 "" H 4500 4650 50  0001 C CNN
+F 2 "Housings_SOIC:SOIC-14_3.9x8.7mm_Pitch1.27mm" H 4500 4650 50  0001 C CNN
 F 3 "" H 4500 4650 50  0000 C CNN
 	3    4500 4650
@@
 F 0 "R38" V 5730 4000 50  0000 C CNN
 F 1 "100" V 5650 4000 50  0000 C CNN
-F 2 "" V 5580 4000 50  0001 C CNN
+F 2 "Resistors_SMD:R_0402" V 5580 4000 50  0001 C CNN
 F 3 "" H 5650 4000 50  0000 C CNN
 	1    5650 4000
@@
 $EndComp
 $Comp
-L +3.3V #PWR069
+L +3.3V #PWR032
 U 1 1 59C7B0E1
 P 5650 3550
-F 0 "#PWR069" H 5650 3400 50  0001 C CNN
+F 0 "#PWR032" H 5650 3400 50  0001 C CNN
 F 1 "+3.3V" H 5650 3690 50  0000 C CNN
 F 2 "" H 5650 3550 50  0000 C CNN
@@
 $EndComp
 $Comp
-L GND #PWR070
+L GND #PWR033
 U 1 1 59C7B28A
 P 5100 3750
-F 0 "#PWR070" H 5100 3500 50  0001 C CNN
+F 0 "#PWR033" H 5100 3500 50  0001 C CNN
 F 1 "GND" H 5100 3600 50  0000 C CNN
 F 2 "" H 5100 3750 50  0000 C CNN
@@
 	4450 2600 4450 2950
 $Comp
-L +3.3V #PWR071
+L +3.3V #PWR034
 U 1 1 59C8723F
 P 4450 2600
-F 0 "#PWR071" H 4450 2450 50  0001 C CNN
+F 0 "#PWR034" H 4450 2450 50  0001 C CNN
 F 1 "+3.3V" H 4450 2740 50  0000 C CNN
 F 2 "" H 4450 2600 50  0000 C CNN
@@
 $EndComp
 $Comp
-L GND #PWR072
+L GND #PWR035
 U 1 1 59C87373
 P 5100 2800
-F 0 "#PWR072" H 5100 2550 50  0001 C CNN
+F 0 "#PWR035" H 5100 2550 50  0001 C CNN
 F 1 "GND" H 5100 2650 50  0000 C CNN
 F 2 "" H 5100 2800 50  0000 C CNN
@@
 	5100 2750 5000 2750
 $Comp
-L GND #PWR073
+L GND #PWR036
 U 1 1 59C8742F
 P 4450 3350
-F 0 "#PWR073" H 4450 3100 50  0001 C CNN
+F 0 "#PWR036" H 4450 3100 50  0001 C CNN
 F 1 "GND" H 4450 3200 50  0000 C CNN
 F 2 "" H 4450 3350 50  0000 C CNN
@@
 TX_DRIVE
 $Comp
-L GND #PWR074
+L GND #PWR037
 U 1 1 59C94C59
 P 2050 6800
-F 0 "#PWR074" H 2050 6550 50  0001 C CNN
+F 0 "#PWR037" H 2050 6550 50  0001 C CNN
 F 1 "GND" H 2050 6650 50  0000 C CNN
 F 2 "" H 2050 6800 50  0000 C CNN
@@
 	2050 6250 2050 6200
 $Comp
-L LED D4
+L LED-RESCUE-interface D4
 U 1 1 59C94C61
 P 2050 6000
+AR Path="/59C94C61" Ref="D4"  Part="1"
+AR Path="/59C7A00B/59C94C61" Ref="D4"  Part="1"
 F 0 "D4" H 2050 6100 50  0000 C CNN
 F 1 "MDB_TX" H 2050 5900 50  0000 C CNN
@@
 F 0 "R35" V 2130 5650 50  0000 C CNN
 F 1 "330" V 2050 5650 50  0000 C CNN
-F 2 "" V 1980 5650 50  0001 C CNN
+F 2 "Resistors_SMD:R_0402" V 1980 5650 50  0001 C CNN
 F 3 "" H 2050 5650 50  0000 C CNN
 	1    2050 5650
@@
 $EndComp
 $Comp
-L +3.3V #PWR075
+L +3.3V #PWR038
 U 1 1 59C94C6F
 P 2050 5500
-F 0 "#PWR075" H 2050 5350 50  0001 C CNN
+F 0 "#PWR038" H 2050 5350 50  0001 C CNN
 F 1 "+3.3V" H 2050 5640 50  0000 C CNN
 F 2 "" H 2050 5500 50  0000 C CNN
@@
 F 0 "Q7" H 2150 6525 50  0000 L CNN
 F 1 "MMBF170" H 2150 6450 50  0000 L CNN
-F 2 "TO_SOT_Packages_SMD:SOT-23" H 2150 6375 50  0000 L CIN
+F 2 "TO_SOT_Packages_SMD:SOT-323_SC-70" H 2150 6375 50  0000 L CIN
 F 3 "" H 1950 6450 50  0000 L CNN
 	1    1950 6450
@@
 RX
 $Comp
-L GND #PWR076
+L GND #PWR039
 U 1 1 59C94D95
 P 4300 6800
-F 0 "#PWR076" H 4300 6550 50  0001 C CNN
+F 0 "#PWR039" H 4300 6550 50  0001 C CNN
 F 1 "GND" H 4300 6650 50  0000 C CNN
 F 2 "" H 4300 6800 50  0000 C CNN
@@
 	4300 6250 4300 6200
 $Comp
-L LED D5
+L LED-RESCUE-interface D5
 U 1 1 59C94D9D
 P 4300 6000
+AR Path="/59C94D9D" Ref="D5"  Part="1"
+AR Path="/59C7A00B/59C94D9D" Ref="D5"  Part="1"
 F 0 "D5" H 4300 6100 50  0000 C CNN
 F 1 "MDB_RX" H 4300 5900 50  0000 C CNN
@@
 F 0 "R36" V 4380 5650 50  0000 C CNN
 F 1 "330" V 4300 5650 50  0000 C CNN
-F 2 "" V 4230 5650 50  0001 C CNN
+F 2 "Resistors_SMD:R_0402" V 4230 5650 50  0001 C CNN
 F 3 "" H 4300 5650 50  0000 C CNN
 	1    4300 5650
@@
 $EndComp
 $Comp
-L +3.3V #PWR077
+L +3.3V #PWR040
 U 1 1 59C94DAB
 P 4300 5500
-F 0 "#PWR077" H 4300 5350 50  0001 C CNN
+F 0 "#PWR040" H 4300 5350 50  0001 C CNN
 F 1 "+3.3V" H 4300 5640 50  0000 C CNN
 F 2 "" H 4300 5500 50  0000 C CNN
@@
 F 0 "Q8" H 4400 6525 50  0000 L CNN
 F 1 "MMBF170" H 4400 6450 50  0000 L CNN
-F 2 "TO_SOT_Packages_SMD:SOT-23" H 4400 6375 50  0000 L CIN
+F 2 "TO_SOT_Packages_SMD:SOT-323_SC-70" H 4400 6375 50  0000 L CIN
 F 3 "" H 4200 6450 50  0000 L CNN
 	1    4200 6450
@@
 F 0 "R40" V 7280 2150 50  0000 C CNN
 F 1 "2.2K" V 7200 2150 50  0000 C CNN
-F 2 "" V 7130 2150 50  0001 C CNN
+F 2 "Resistors_SMD:R_0402" V 7130 2150 50  0001 C CNN
 F 3 "" H 7200 2150 50  0000 C CNN
 	1    7200 2150
@@
 F 0 "W14" H 3200 4820 50  0000 C CNN
 F 1 "RX" H 3200 4750 50  0000 C CNN
-F 2 "" H 3400 4550 50  0001 C CNN
+F 2 "Measurement_Points:Test_Point" H 3400 4550 50  0001 C CNN
 F 3 "" H 3400 4550 50  0000 C CNN
 	1    3200 4550
@@
 F 0 "W13" H 3200 3220 50  0000 C CNN
 F 1 "TX" H 3200 3150 50  0000 C CNN
-F 2 "" H 3400 2950 50  0001 C CNN
+F 2 "Measurement_Points:Test_Point" H 3400 2950 50  0001 C CNN
 F 3 "" H 3400 2950 50  0000 C CNN
 	1    3200 2950
@@
 F 0 "W12" H 3200 2420 50  0000 C CNN
 F 1 "POW" H 3200 2350 50  0000 C CNN
-F 2 "" H 3400 2150 50  0001 C CNN
+F 2 "Measurement_Points:Test_Point" H 3400 2150 50  0001 C CNN
 F 3 "" H 3400 2150 50  0000 C CNN
 	1    3200 2150
@@
 F 0 "W16" H 5650 4570 50  0000 C CNN
 F 1 "RX_IN" H 5650 4500 50  0000 C CNN
-F 2 "" H 5850 4300 50  0001 C CNN
+F 2 "Measurement_Points:Test_Point" H 5850 4300 50  0001 C CNN
 F 3 "" H 5850 4300 50  0000 C CNN
 	1    5650 4300
@@
 F 0 "W15" H 5400 3020 50  0000 C CNN
 F 1 "TX_LED" H 5400 2950 50  0000 C CNN
-F 2 "" H 5600 2750 50  0001 C CNN
+F 2 "Measurement_Points:Test_Point" H 5600 2750 50  0001 C CNN
 F 3 "" H 5600 2750 50  0000 C CNN
 	1    5400 2750
@@
 NoConn ~ 6250 3950
 $Comp
-L Jumper_NO_Small JP?
+L Jumper_NO_Small JP2
 U 1 1 5A273710
 P 5850 2450
-F 0 "JP?" H 5850 2530 50  0000 C CNN
+F 0 "JP2" H 5850 2530 50  0000 C CNN
 F 1 "Jumper_NO_Small" H 5860 2390 50  0001 C CNN
-F 2 "" H 5850 2450 50  0000 C CNN
+F 2 "" H 5850 2450 50  0001 C CNN
 F 3 "" H 5850 2450 50  0000 C CNN
 	1    5850 2450

Commit message: Start of layout
Parts:
- D6: footprint (none) -> Diodes_SMD:SMA_Handsoldering
- JP2: footprint (none) -> Resistors_SMD:R_0402
- Q7, Q8: footprint TO_SOT_Packages_SMD:SOT-323_SC-70 -> TO_SOT_Packages_SMD:SC-70
- U5, U6: footprint Housings_DIP:DIP-6_W7.62mm_Socket -> Housings_DIP:DIP-6_W7.62mm; symbol 4N25 -> 4N25-RESCUE-interface
- U7: footprint Housings_DIP:DIP-8_W7.62mm_Socket -> Housings_DIP:DIP-8_W7.62mm; symbol 6N136 -> 6N136-RESCUE-interface
Connections:
- net TX_DRIVE: now also R39.2, U4.2, W15.1
Changed lines of the file:
@@
 $EndDescr
 $Comp
-L 4N25 U6
+L 4N25-RESCUE-interface U6
 U 1 1 59C7A067
 P 6550 3150
 F 0 "U6" H 6350 3350 50  0000 L CNN
 F 1 "4N29" H 6550 3350 50  0000 L CNN
-F 2 "Housings_DIP:DIP-6_W7.62mm_Socket" H 6350 2950 50  0000 L CIN
+F 2 "Housings_DIP:DIP-6_W7.62mm" H 6350 2950 50  0000 L CIN
 F 3 "" H 6550 3150 50  0000 L CNN
 	1    6550 3150
@@
 $EndComp
 $Comp
-L 4N25 U5
+L 4N25-RESCUE-interface U5
 U 1 1 59C7A083
 P 6550 2250
 F 0 "U5" H 6350 2450 50  0000 L CNN
 F 1 "4N29" H 6550 2450 50  0000 L CNN
-F 2 "Housings_DIP:DIP-6_W7.62mm_Socket" H 6350 2050 50  0000 L CIN
+F 2 "Housings_DIP:DIP-6_W7.62mm" H 6350 2050 50  0000 L CIN
 F 3 "" H 6550 2250 50  0000 L CNN
 	1    6550 2250
@@
 $EndComp
 $Comp
-L 6N136 U7
+L 6N136-RESCUE-interface U7
 U 1 1 59C7A155
 P 6550 4050
 F 0 "U7" H 6350 4350 50  0000 L CNN
 F 1 "6N137" H 6550 4350 50  0000 L CNN
-F 2 "Housings_DIP:DIP-8_W7.62mm_Socket" H 6350 3750 50  0000 L CIN
+F 2 "Housings_DIP:DIP-8_W7.62mm" H 6350 3750 50  0000 L CIN
 F 3 "" H 6550 4050 50  0000 L CNN
 	1    6550 4050
@@
 F 0 "D6" H 7450 2600 50  0000 C CNN
 F 1 "TVS" H 7450 2400 50  0000 C CNN
-F 2 "" H 7450 2500 50  0001 C CNN
+F 2 "Diodes_SMD:SMA_Handsoldering" H 7450 2500 50  0001 C CNN
 F 3 "" H 7450 2500 50  0000 C CNN
 	1    7450 2500
@@
 $EndComp
 $Comp
-L +3.3V #PWR030
+L +3.3V #PWR36
 U 1 1 59C7A9C9
 P 4850 1550
-F 0 "#PWR030" H 4850 1400 50  0001 C CNN
+F 0 "#PWR36" H 4850 1400 50  0001 C CNN
 F 1 "+3.3V" H 4850 1690 50  0000 C CNN
 F 2 "" H 4850 1550 50  0000 C CNN
@@
 LOW when the vending \nmachine is powered.
 $Comp
-L GND #PWR031
+L GND #PWR40
 U 1 1 59C7AA95
 P 6050 4400
-F 0 "#PWR031" H 6050 4150 50  0001 C CNN
+F 0 "#PWR40" H 6050 4150 50  0001 C CNN
 F 1 "GND" H 6050 4250 50  0000 C CNN
 F 2 "" H 6050 4400 50  0000 C CNN
@@
 $EndComp
 $Comp
-L +3.3V #PWR032
+L +3.3V #PWR39
 U 1 1 59C7B0E1
 P 5650 3550
-F 0 "#PWR032" H 5650 3400 50  0001 C CNN
+F 0 "#PWR39" H 5650 3400 50  0001 C CNN
 F 1 "+3.3V" H 5650 3690 50  0000 C CNN
 F 2 "" H 5650 3550 50  0000 C CNN
@@
 $EndComp
 $Comp
-L GND #PWR033
+L GND #PWR38
 U 1 1 59C7B28A
 P 5100 3750
-F 0 "#PWR033" H 5100 3500 50  0001 C CNN
+F 0 "#PWR38" H 5100 3500 50  0001 C CNN
 F 1 "GND" H 5100 3600 50  0000 C CNN
 F 2 "" H 5100 3750 50  0000 C CNN
@@
 	4450 2600 4450 2950
 $Comp
-L +3.3V #PWR034
+L +3.3V #PWR34
 U 1 1 59C8723F
 P 4450 2600
-F 0 "#PWR034" H 4450 2450 50  0001 C CNN
+F 0 "#PWR34" H 4450 2450 50  0001 C CNN
 F 1 "+3.3V" H 4450 2740 50  0000 C CNN
 F 2 "" H 4450 2600 50  0000 C CNN
@@
 $EndComp
 $Comp
-L GND #PWR035
+L GND #PWR37
 U 1 1 59C87373
 P 5100 2800
-F 0 "#PWR035" H 5100 2550 50  0001 C CNN
+F 0 "#PWR37" H 5100 2550 50  0001 C CNN
 F 1 "GND" H 5100 2650 50  0000 C CNN
 F 2 "" H 5100 2800 50  0000 C CNN
@@
 	5100 2750 5000 2750
 $Comp
-L GND #PWR036
+L GND #PWR35
 U 1 1 59C8742F
 P 4450 3350
-F 0 "#PWR036" H 4450 3100 50  0001 C CNN
+F 0 "#PWR35" H 4450 3100 50  0001 C CNN
 F 1 "GND" H 4450 3200 50  0000 C CNN
 F 2 "" H 4450 3350 50  0000 C CNN
@@
 	1    0    0    -1
 $EndComp
-Text Label 4950 3150 0    59   ~ 0
+Text Label 5000 3050 0    59   ~ 0
 TX_DRIVE
 Text Label 4950 4400 0    59   ~ 0
@@
 TX_DRIVE
 $Comp
-L GND #PWR037
+L GND #PWR31
 U 1 1 59C94C59
 P 2050 6800
-F 0 "#PWR037" H 2050 6550 50  0001 C CNN
+F 0 "#PWR31" H 2050 6550 50  0001 C CNN
 F 1 "GND" H 2050 6650 50  0000 C CNN
 F 2 "" H 2050 6800 50  0000 C CNN
@@
 $EndComp
 $Comp
-L +3.3V #PWR038
+L +3.3V #PWR30
 U 1 1 59C94C6F
 P 2050 5500
-F 0 "#PWR038" H 2050 5350 50  0001 C CNN
+F 0 "#PWR30" H 2050 5350 50  0001 C CNN
 F 1 "+3.3V" H 2050 5640 50  0000 C CNN
 F 2 "" H 2050 5500 50  0000 C CNN
@@
 F 0 "Q7" H 2150 6525 50  0000 L CNN
 F 1 "MMBF170" H 2150 6450 50  0000 L CNN
-F 2 "TO_SOT_Packages_SMD:SOT-323_SC-70" H 2150 6375 50  0000 L CIN
+F 2 "TO_SOT_Packages_SMD:SC-70" H 2150 6375 50  0000 L CIN
 F 3 "" H 1950 6450 50  0000 L CNN
 	1    1950 6450
@@
 RX
 $Comp
-L GND #PWR039
+L GND #PWR33
 U 1 1 59C94D95
 P 4300 6800
-F 0 "#PWR039" H 4300 6550 50  0001 C CNN
+F 0 "#PWR33" H 4300 6550 50  0001 C CNN
 F 1 "GND" H 4300 6650 50  0000 C CNN
 F 2 "" H 4300 6800 50  0000 C CNN
@@
 $EndComp
 $Comp
-L +3.3V #PWR040
+L +3.3V #PWR32
 U 1 1 59C94DAB
 P 4300 5500
-F 0 "#PWR040" H 4300 5350 50  0001 C CNN
+F 0 "#PWR32" H 4300 5350 50  0001 C CNN
 F 1 "+3.3V" H 4300 5640 50  0000 C CNN
 F 2 "" H 4300 5500 50  0000 C CNN
@@
 F 0 "Q8" H 4400 6525 50  0000 L CNN
 F 1 "MMBF170" H 4400 6450 50  0000 L CNN
-F 2 "TO_SOT_Packages_SMD:SOT-323_SC-70" H 4400 6375 50  0000 L CIN
+F 2 "TO_SOT_Packages_SMD:SC-70" H 4400 6375 50  0000 L CIN
 F 3 "" H 4200 6450 50  0000 L CNN
 	1    4200 6450
@@
 F 0 "JP2" H 5850 2530 50  0000 C CNN
 F 1 "Jumper_NO_Small" H 5860 2390 50  0001 C CNN
-F 2 "" H 5850 2450 50  0001 C CNN
+F 2 "Resistors_SMD:R_0402" H 5850 2450 50  0001 C CNN
 F 3 "" H 5850 2450 50  0000 C CNN
 	1    5850 2450
