File: interface/pcb/power.sch (KiCad schematic (older format))
At the start: 21 parts, among them J1 2.1MM BARREL, P6 POWER OUT, Q9 DMP3099, U10 AP1509-50, U9 AP1509-33

Commit message: PCB revisions
Parts:
- removed C24: 22uF, Capacitors_SMD:c_elec_5x5.3, symbol CP
- removed C26: 0.1uF, Capacitors_SMD:C_0402, symbol C
- removed D9: D_Schottky, symbol D_Schottky
- removed F3: 1A, symbol Polyfuse
- removed L2: 47uH, symbol INDUCTOR_SMALL
- removed U10: AP1509-50, symbol AP1509
Connections:
- net labels removed: +5V
- wire segments 64 -> 41
- no-connect marks 0 -> 1
Other:
- moved on the sheet: P6

Commit message: Partial BOM
Parts:
- C21, C22: footprint Capacitors_SMD:c_elec_6.3x5.3 -> Capacitors_SMD:CP_Elec_6.3x5.3
- C23: footprint Capacitors_SMD:c_elec_5x5.3 -> Capacitors_SMD:CP_Elec_5x5.3
- D7: symbol LED -> LED-RESCUE-interface
- U9: footprint (none) -> Housings_SOIC:SOIC-8_3.9x4.9mm_Pitch1.27mm
- gave numbers to parts that had none: 1
Other:
- note added: "Seeed SKU 303010168"
Changed lines of the file:
@@
 EESchema Schematic File Version 2
+LIBS:interface-rescue
 LIBS:power
 LIBS:device
@@
 LIBS:tpd4s012
 LIBS:ap1509
-LIBS:device_big
 LIBS:SeeedOPL-Resistor-2016
 LIBS:SeeedOPL-Connector-2016
 LIBS:SeeedOPL-Inductor-2016
 LIBS:SeeedOPL-Display-2016
+LIBS:nhd-c0220biz
 LIBS:interface-cache
 EELAYER 25 0
@@
 Connection ~ 3200 3200
 $Comp
-L GND #PWR091
+L GND #PWR041
 U 1 1 59C93412
 P 3200 3500
-F 0 "#PWR091" H 3200 3250 50  0001 C CNN
+F 0 "#PWR041" H 3200 3250 50  0001 C CNN
 F 1 "GND" H 3200 3350 50  0000 C CNN
 F 2 "" H 3200 3500 50  0000 C CNN
@@
 	4150 2550 4150 2950
 $Comp
-L +12V #PWR092
+L +12V #PWR042
 U 1 1 59C9341A
 P 4150 2050
-F 0 "#PWR092" H 4150 1900 50  0001 C CNN
+F 0 "#PWR042" H 4150 1900 50  0001 C CNN
 F 1 "+12V" H 4150 2190 50  0000 C CNN
 F 2 "" H 4150 2050 50  0000 C CNN
@@
 F 0 "C21" H 4175 3200 50  0000 L CNN
 F 1 "47uF" H 4175 3000 50  0000 L CNN
-F 2 "Capacitors_SMD:c_elec_6.3x5.3" H 4188 2950 50  0001 C CNN
+F 2 "Capacitors_SMD:CP_Elec_6.3x5.3" H 4188 2950 50  0001 C CNN
 F 3 "" H 4150 3100 50  0000 C CNN
 	1    4150 3100
@@
 	4150 3250 4150 3500
 $Comp
-L GND #PWR093
+L GND #PWR043
 U 1 1 59C93429
 P 4150 3500
-F 0 "#PWR093" H 4150 3250 50  0001 C CNN
+F 0 "#PWR043" H 4150 3250 50  0001 C CNN
 F 1 "GND" H 4150 3350 50  0000 C CNN
 F 2 "" H 4150 3500 50  0000 C CNN
@@
 F 0 "U9" H 6300 2600 60  0000 C CNN
 F 1 "AP1509-33" H 6300 3300 60  0000 C CNN
-F 2 "" H 6300 2950 60  0001 C CNN
+F 2 "Housings_SOIC:SOIC-8_3.9x4.9mm_Pitch1.27mm" H 6300 2950 60  0001 C CNN
 F 3 "" H 6300 2950 60  0000 C CNN
 	1    6300 2950
@@
 	5900 2950 5750 2950
 $Comp
-L GND #PWR094
+L GND #PWR044
 U 1 1 59C93443
 P 5750 3500
-F 0 "#PWR094" H 5750 3250 50  0001 C CNN
+F 0 "#PWR044" H 5750 3250 50  0001 C CNN
 F 1 "GND" H 5750 3350 50  0000 C CNN
 F 2 "" H 5750 3500 50  0000 C CNN
@@
 $EndComp
 $Comp
-L GND #PWR095
+L GND #PWR045
 U 1 1 59C93449
 P 6800 3500
-F 0 "#PWR095" H 6800 3250 50  0001 C CNN
+F 0 "#PWR045" H 6800 3250 50  0001 C CNN
 F 1 "GND" H 6800 3350 50  0000 C CNN
 F 2 "" H 6800 3500 50  0000 C CNN
@@
 	7150 3350 7150 3500
 $Comp
-L GND #PWR096
+L GND #PWR046
 U 1 1 59C93461
 P 7150 3500
-F 0 "#PWR096" H 7150 3250 50  0001 C CNN
+F 0 "#PWR046" H 7150 3250 50  0001 C CNN
 F 1 "GND" H 7150 3350 50  0000 C CNN
 F 2 "" H 7150 3500 50  0000 C CNN
@@
 F 0 "C23" H 7925 3300 50  0000 L CNN
 F 1 "22uF" H 7925 3100 50  0000 L CNN
-F 2 "Capacitors_SMD:c_elec_5x5.3" H 7938 3050 50  0001 C CNN
+F 2 "Capacitors_SMD:CP_Elec_5x5.3" H 7938 3050 50  0001 C CNN
 F 3 "" H 7900 3200 50  0000 C CNN
 	1    7900 3200
@@
 	7900 3350 7900 3500
 $Comp
-L GND #PWR097
+L GND #PWR047
 U 1 1 59C93473
 P 7900 3500
-F 0 "#PWR097" H 7900 3250 50  0001 C CNN
+F 0 "#PWR047" H 7900 3250 50  0001 C CNN
 F 1 "GND" H 7900 3350 50  0000 C CNN
 F 2 "" H 7900 3500 50  0000 C CNN
@@
 	8250 3350 8250 3500
 $Comp
-L GND #PWR098
+L GND #PWR048
 U 1 1 59C93486
 P 8250 3500
-F 0 "#PWR098" H 8250 3250 50  0001 C CNN
+F 0 "#PWR048" H 8250 3250 50  0001 C CNN
 F 1 "GND" H 8250 3350 50  0000 C CNN
 F 2 "" H 8250 3500 50  0000 C CNN
@@
 $EndComp
 $Comp
-L +3.3V #PWR099
+L +3.3V #PWR049
 U 1 1 59C9348C
 P 8950 2550
-F 0 "#PWR099" H 8950 2400 50  0001 C CNN
+F 0 "#PWR049" H 8950 2400 50  0001 C CNN
 F 1 "+3.3V" H 8950 2690 50  0000 C CNN
 F 2 "" H 8950 2550 50  0000 C CNN
@@
 F 0 "C22" H 4475 3200 50  0000 L CNN
 F 1 "47uF" H 4475 3000 50  0000 L CNN
-F 2 "Capacitors_SMD:c_elec_6.3x5.3" H 4488 2950 50  0001 C CNN
+F 2 "Capacitors_SMD:CP_Elec_6.3x5.3" H 4488 2950 50  0001 C CNN
 F 3 "" H 4450 3100 50  0000 C CNN
 	1    4450 3100
@@
 	4450 3250 4450 3500
 $Comp
-L GND #PWR0100
+L GND #PWR050
 U 1 1 59C9349C
 P 4450 3500
-F 0 "#PWR0100" H 4450 3250 50  0001 C CNN
+F 0 "#PWR050" H 4450 3250 50  0001 C CNN
 F 1 "GND" H 4450 3350 50  0000 C CNN
 F 2 "" H 4450 3500 50  0000 C CNN
@@
 	4150 2050 4150 2250
 $Comp
-L LED D7
+L LED-RESCUE-interface D7
 U 1 1 59C945E1
 P 3850 4750
+AR Path="/59C945E1" Ref="D7"  Part="1"
+AR Path="/59C92DEF/59C945E1" Ref="D7"  Part="1"
 F 0 "D7" H 3850 4850 50  0000 C CNN
 F 1 "POWER" H 3850 4650 50  0000 C CNN
@@
 $EndComp
 $Comp
-L GND #PWR0107
+L GND #PWR051
 U 1 1 59C94770
 P 3850 4950
-F 0 "#PWR0107" H 3850 4700 50  0001 C CNN
+F 0 "#PWR051" H 3850 4700 50  0001 C CNN
 F 1 "GND" H 3850 4800 50  0000 C CNN
 F 2 "" H 3850 4950 50  0000 C CNN
@@
 	7750 4800 7750 5150
 $Comp
-L GND #PWR0108
+L GND #PWR052
 U 1 1 59C993CF
 P 7750 5150
-F 0 "#PWR0108" H 7750 4900 50  0001 C CNN
+F 0 "#PWR052" H 7750 4900 50  0001 C CNN
 F 1 "GND" H 7750 5000 50  0000 C CNN
 F 2 "" H 7750 5150 50  0000 C CNN
@@
 $EndComp
 $Comp
-L +3.3V #PWR0110
+L +3.3V #PWR053
 U 1 1 59C99499
 P 7150 4300
-F 0 "#PWR0110" H 7150 4150 50  0001 C CNN
+F 0 "#PWR053" H 7150 4150 50  0001 C CNN
 F 1 "+3.3V" H 7150 4440 50  0000 C CNN
 F 2 "" H 7150 4300 50  0000 C CNN
@@
 $EndComp
 $Comp
-L +12V #PWR0111
+L +12V #PWR054
 U 1 1 59C99508
 P 7250 4450
-F 0 "#PWR0111" H 7250 4300 50  0001 C CNN
+F 0 "#PWR054" H 7250 4300 50  0001 C CNN
 F 1 "+12V" H 7250 4590 50  0000 C CNN
 F 2 "" H 7250 4450 50  0000 C CNN
@@
 320120003
 $Comp
-L C C?
+L C C18
 U 1 1 5A00AB29
 P 4750 3100
-F 0 "C?" H 4775 3200 50  0000 L CNN
+F 0 "C18" H 4775 3200 50  0000 L CNN
 F 1 "0.1uF" H 4775 3000 50  0000 L CNN
 F 2 "Capacitors_SMD:C_0402" H 4788 2950 50  0001 C CNN
@@
 	4750 3250 4750 3500
 $Comp
-L GND #PWR?
+L GND #PWR055
 U 1 1 5A00ACB2
 P 4750 3500
-F 0 "#PWR?" H 4750 3250 50  0001 C CNN
+F 0 "#PWR055" H 4750 3250 50  0001 C CNN
 F 1 "GND" H 4750 3350 50  0000 C CNN
 F 2 "" H 4750 3500 50  0000 C CNN
@@
 $EndComp
 NoConn ~ 7350 4900
+Text Notes 7200 2550 0    30   ~ 0
+Seeed SKU 303010168
 $EndSCHEMATC

Commit message: Start of layout
Parts:
- C21, C22: footprint Capacitors_SMD:CP_Elec_6.3x5.3 -> Capacitors_SMD:c_elec_6.3x7.7
- C23: footprint Capacitors_SMD:CP_Elec_5x5.3 -> Capacitors_SMD:c_elec_5x5.3
- D8: footprint (none) -> Diodes_SMD:SMA_Handsoldering
- F1, F2: footprint (none) -> SeeedOPL-Fuse-2016:F1812
- J1: footprint (none) -> SeeedOPL-Connector-2016:DCJ3P-14.2X11.0X9.0MM
- L1: footprint (none) -> Inductor_SMD:L_12x12mm_h6mm
- P6: footprint (none) -> Sockets_MOLEX_KK-System:Socket_MOLEX-KK-RM2-54mm_Lock_4pin_straight
- Q9: footprint (none) -> TO_SOT_Packages_SMD:SOT-23
- R45: footprint (none) -> Resistors_SMD:R_0402
Changed lines of the file:
@@
 F 0 "Q9" V 3950 2900 50  0000 R CNN
 F 1 "DMP3099" V 3850 2900 50  0000 R CNN
-F 2 "" H 3850 2950 50  0001 C CNN
+F 2 "TO_SOT_Packages_SMD:SOT-23" H 3850 2950 50  0001 C CNN
 F 3 "" H 3650 2850 50  0000 C CNN
 	1    3650 2850
@@
 Connection ~ 3200 3200
 $Comp
-L GND #PWR041
+L GND #PWR41
 U 1 1 59C93412
 P 3200 3500
-F 0 "#PWR041" H 3200 3250 50  0001 C CNN
+F 0 "#PWR41" H 3200 3250 50  0001 C CNN
 F 1 "GND" H 3200 3350 50  0000 C CNN
 F 2 "" H 3200 3500 50  0000 C CNN
@@
 	4150 2550 4150 2950
 $Comp
-L +12V #PWR042
+L +12V #PWR43
 U 1 1 59C9341A
 P 4150 2050
-F 0 "#PWR042" H 4150 1900 50  0001 C CNN
+F 0 "#PWR43" H 4150 1900 50  0001 C CNN
 F 1 "+12V" H 4150 2190 50  0000 C CNN
 F 2 "" H 4150 2050 50  0000 C CNN
@@
 F 0 "C21" H 4175 3200 50  0000 L CNN
 F 1 "47uF" H 4175 3000 50  0000 L CNN
-F 2 "Capacitors_SMD:CP_Elec_6.3x5.3" H 4188 2950 50  0001 C CNN
+F 2 "Capacitors_SMD:c_elec_6.3x7.7" H 4188 2950 50  0001 C CNN
 F 3 "" H 4150 3100 50  0000 C CNN
 	1    4150 3100
@@
 	4150 3250 4150 3500
 $Comp
-L GND #PWR043
+L GND #PWR44
 U 1 1 59C93429
 P 4150 3500
-F 0 "#PWR043" H 4150 3250 50  0001 C CNN
+F 0 "#PWR44" H 4150 3250 50  0001 C CNN
 F 1 "GND" H 4150 3350 50  0000 C CNN
 F 2 "" H 4150 3500 50  0000 C CNN
@@
 	5900 2950 5750 2950
 $Comp
-L GND #PWR044
+L GND #PWR47
 U 1 1 59C93443
 P 5750 3500
-F 0 "#PWR044" H 5750 3250 50  0001 C CNN
+F 0 "#PWR47" H 5750 3250 50  0001 C CNN
 F 1 "GND" H 5750 3350 50  0000 C CNN
 F 2 "" H 5750 3500 50  0000 C CNN
@@
 $EndComp
 $Comp
-L GND #PWR045
+L GND #PWR48
 U 1 1 59C93449
 P 6800 3500
-F 0 "#PWR045" H 6800 3250 50  0001 C CNN
+F 0 "#PWR48" H 6800 3250 50  0001 C CNN
 F 1 "GND" H 6800 3350 50  0000 C CNN
 F 2 "" H 6800 3500 50  0000 C CNN
@@
 F 0 "L1" H 7500 2850 50  0000 C CNN
 F 1 "47uH" H 7500 2700 50  0000 C CNN
-F 2 "" H 7500 2750 50  0001 C CNN
+F 2 "Inductor_SMD:L_12x12mm_h6mm" H 7500 2750 50  0001 C CNN
 F 3 "" H 7500 2750 50  0000 C CNN
 	1    7500 2750
@@
 F 0 "D8" H 7150 3300 50  0000 C CNN
 F 1 "D_Schottky" H 7150 3100 50  0000 C CNN
-F 2 "" H 7150 3200 50  0001 C CNN
+F 2 "Diodes_SMD:SMA_Handsoldering" H 7150 3200 50  0001 C CNN
 F 3 "" H 7150 3200 50  0000 C CNN
 	1    7150 3200
@@
 	7150 3350 7150 3500
 $Comp
-L GND #PWR046
+L GND #PWR49
 U 1 1 59C93461
 P 7150 3500
-F 0 "#PWR046" H 7150 3250 50  0001 C CNN
+F 0 "#PWR49" H 7150 3250 50  0001 C CNN
 F 1 "GND" H 7150 3350 50  0000 C CNN
 F 2 "" H 7150 3500 50  0000 C CNN
@@
 F 0 "C23" H 7925 3300 50  0000 L CNN
 F 1 "22uF" H 7925 3100 50  0000 L CNN
-F 2 "Capacitors_SMD:CP_Elec_5x5.3" H 7938 3050 50  0001 C CNN
+F 2 "Capacitors_SMD:c_elec_5x5.3" H 7938 3050 50  0001 C CNN
 F 3 "" H 7900 3200 50  0000 C CNN
 	1    7900 3200
@@
 	7900 3350 7900 3500
 $Comp
-L GND #PWR047
+L GND #PWR53
 U 1 1 59C93473
 P 7900 3500
-F 0 "#PWR047" H 7900 3250 50  0001 C CNN
+F 0 "#PWR53" H 7900 3250 50  0001 C CNN
 F 1 "GND" H 7900 3350 50  0000 C CNN
 F 2 "" H 7900 3500 50  0000 C CNN
@@
 	8250 3350 8250 3500
 $Comp
-L GND #PWR048
+L GND #PWR54
 U 1 1 59C93486
 P 8250 3500
-F 0 "#PWR048" H 8250 3250 50  0001 C CNN
+F 0 "#PWR54" H 8250 3250 50  0001 C CNN
 F 1 "GND" H 8250 3350 50  0000 C CNN
 F 2 "" H 8250 3500 50  0000 C CNN
@@
 $EndComp
 $Comp
-L +3.3V #PWR049
+L +3.3V #PWR55
 U 1 1 59C9348C
 P 8950 2550
-F 0 "#PWR049" H 8950 2400 50  0001 C CNN
+F 0 "#PWR55" H 8950 2400 50  0001 C CNN
 F 1 "+3.3V" H 8950 2690 50  0000 C CNN
 F 2 "" H 8950 2550 50  0000 C CNN
@@
 F 0 "C22" H 4475 3200 50  0000 L CNN
 F 1 "47uF" H 4475 3000 50  0000 L CNN
-F 2 "Capacitors_SMD:CP_Elec_6.3x5.3" H 4488 2950 50  0001 C CNN
+F 2 "Capacitors_SMD:c_elec_6.3x7.7" H 4488 2950 50  0001 C CNN
 F 3 "" H 4450 3100 50  0000 C CNN
 	1    4450 3100
@@
 	4450 3250 4450 3500
 $Comp
-L GND #PWR050
+L GND #PWR45
 U 1 1 59C9349C
 P 4450 3500
-F 0 "#PWR050" H 4450 3250 50  0001 C CNN
+F 0 "#PWR45" H 4450 3250 50  0001 C CNN
 F 1 "GND" H 4450 3350 50  0000 C CNN
 F 2 "" H 4450 3500 50  0000 C CNN
@@
 F 0 "F2" V 8550 2750 50  0000 C CNN
 F 1 "1A" V 8750 2750 50  0000 C CNN
-F 2 "" H 8700 2550 50  0001 L CNN
+F 2 "SeeedOPL-Fuse-2016:F1812" H 8700 2550 50  0001 L CNN
 F 3 "" H 8650 2750 50  0001 C CNN
 	1    8650 2750
@@
 F 0 "F1" V 4050 2400 50  0000 C CNN
 F 1 "1A" V 4250 2400 50  0000 C CNN
-F 2 "" H 4200 2200 50  0001 L CNN
+F 2 "SeeedOPL-Fuse-2016:F1812" H 4200 2200 50  0001 L CNN
 F 3 "" H 4150 2400 50  0001 C CNN
 	1    4150 2400
@@
 $EndComp
 $Comp
-L GND #PWR051
+L GND #PWR42
 U 1 1 59C94770
 P 3850 4950
-F 0 "#PWR051" H 3850 4700 50  0001 C CNN
+F 0 "#PWR42" H 3850 4700 50  0001 C CNN
 F 1 "GND" H 3850 4800 50  0000 C CNN
 F 2 "" H 3850 4950 50  0000 C CNN
@@
 F 0 "R45" V 3930 4400 50  0000 C CNN
 F 1 "1.5K" V 3850 4400 50  0000 C CNN
-F 2 "" V 3780 4400 50  0001 C CNN
+F 2 "Resistors_SMD:R_0402" V 3780 4400 50  0001 C CNN
 F 3 "" H 3850 4400 50  0000 C CNN
 	1    3850 4400
@@
 F 0 "P6" H 7300 5350 50  0000 C CNN
 F 1 "POWER OUT" V 7400 5100 50  0000 C CNN
-F 2 "" H 7300 5100 50  0001 C CNN
+F 2 "Sockets_MOLEX_KK-System:Socket_MOLEX-KK-RM2-54mm_Lock_4pin_straight" H 7300 5100 50  0001 C CNN
 F 3 "" H 7300 5100 50  0000 C CNN
 	1    7300 5100
@@
 	7750 4800 7750 5150
 $Comp
-L GND #PWR052
+L GND #PWR52
 U 1 1 59C993CF
 P 7750 5150
-F 0 "#PWR052" H 7750 4900 50  0001 C CNN
+F 0 "#PWR52" H 7750 4900 50  0001 C CNN
 F 1 "GND" H 7750 5000 50  0000 C CNN
 F 2 "" H 7750 5150 50  0000 C CNN
@@
 $EndComp
 $Comp
-L +3.3V #PWR053
+L +3.3V #PWR50
 U 1 1 59C99499
 P 7150 4300
-F 0 "#PWR053" H 7150 4150 50  0001 C CNN
+F 0 "#PWR50" H 7150 4150 50  0001 C CNN
 F 1 "+3.3V" H 7150 4440 50  0000 C CNN
 F 2 "" H 7150 4300 50  0000 C CNN
@@
 $EndComp
 $Comp
-L +12V #PWR054
+L +12V #PWR51
 U 1 1 59C99508
 P 7250 4450
-F 0 "#PWR054" H 7250 4300 50  0001 C CNN
+F 0 "#PWR51" H 7250 4300 50  0001 C CNN
 F 1 "+12V" H 7250 4590 50  0000 C CNN
 F 2 "" H 7250 4450 50  0000 C CNN
@@
 F 0 "J1" H 2350 3050 45  0000 L BNN
 F 1 "2.1MM BARREL" H 2600 3050 45  0000 L BNN
-F 2 "" H 2550 2850 79  0001 C CNN
+F 2 "SeeedOPL-Connector-2016:DCJ3P-14.2X11.0X9.0MM" H 2550 2850 79  0001 C CNN
 F 3 "" H 2550 2850 79  0000 C CNN
 F 4 "320120003" H 2580 3000 20  0001 C CNN "SKU"
@@
 	4750 3250 4750 3500
 $Comp
-L GND #PWR055
+L GND #PWR46
 U 1 1 5A00ACB2
 P 4750 3500
-F 0 "#PWR055" H 4750 3250 50  0001 C CNN
+F 0 "#PWR46" H 4750 3250 50  0001 C CNN
 F 1 "GND" H 4750 3350 50  0000 C CNN
 F 2 "" H 4750 3500 50  0000 C CNN
