File: interface/pcb/sdcard.sch (KiCad schematic (older format))
At the start: 15 parts, among them Q1 MMBF170

Commit message: Partial BOM
Parts:
- D1: symbol LED -> LED-RESCUE-interface
- Q1: footprint TO_SOT_Packages_SMD:SOT-23 -> TO_SOT_Packages_SMD:SOT-323_SC-70
- R1, R2, R3, R4, R5, R6: footprint (none) -> Resistors_SMD:R_0402
- W1, W2, W3, W4, W5: footprint (none) -> Measurement_Points:Test_Point
Changed lines of the file:
@@
 EESchema Schematic File Version 2
+LIBS:interface-rescue
 LIBS:power
 LIBS:device
@@
 LIBS:tpd4s012
 LIBS:ap1509
-LIBS:device_big
 LIBS:SeeedOPL-Resistor-2016
 LIBS:SeeedOPL-Connector-2016
 LIBS:SeeedOPL-Inductor-2016
 LIBS:SeeedOPL-Display-2016
+LIBS:nhd-c0220biz
 LIBS:interface-cache
 EELAYER 25 0
@@
 F 0 "W1" H 3800 3020 50  0000 C CNN
 F 1 "CS" H 3800 2950 50  0000 C CNN
-F 2 "" H 4000 2750 50  0001 C CNN
+F 2 "Measurement_Points:Test_Point" H 4000 2750 50  0001 C CNN
 F 3 "" H 4000 2750 50  0000 C CNN
 	1    3800 2750
@@
 F 0 "W2" H 4000 3020 50  0000 C CNN
 F 1 "MOSI" H 4000 2950 50  0000 C CNN
-F 2 "" H 4200 2750 50  0001 C CNN
+F 2 "Measurement_Points:Test_Point" H 4200 2750 50  0001 C CNN
 F 3 "" H 4200 2750 50  0000 C CNN
 	1    4000 2750
@@
 F 0 "W3" H 4200 3020 50  0000 C CNN
 F 1 "SCK" H 4200 2950 50  0000 C CNN
-F 2 "" H 4400 2750 50  0001 C CNN
+F 2 "Measurement_Points:Test_Point" H 4400 2750 50  0001 C CNN
 F 3 "" H 4400 2750 50  0000 C CNN
 	1    4200 2750
@@
 F 0 "W4" H 4400 3020 50  0000 C CNN
 F 1 "MISO" H 4400 2950 50  0000 C CNN
-F 2 "" H 4600 2750 50  0001 C CNN
+F 2 "Measurement_Points:Test_Point" H 4600 2750 50  0001 C CNN
 F 3 "" H 4600 2750 50  0000 C CNN
 	1    4400 2750
@@
 F 0 "R4" V 5380 3250 50  0000 C CNN
 F 1 "22" V 5300 3250 50  0000 C CNN
-F 2 "" V 5230 3250 50  0001 C CNN
+F 2 "Resistors_SMD:R_0402" V 5230 3250 50  0001 C CNN
 F 3 "" H 5300 3250 50  0000 C CNN
 	1    5300 3250
@@
 F 0 "R2" V 4980 3350 50  0000 C CNN
 F 1 "22" V 4900 3350 50  0000 C CNN
-F 2 "" V 4830 3350 50  0001 C CNN
+F 2 "Resistors_SMD:R_0402" V 4830 3350 50  0001 C CNN
 F 3 "" H 4900 3350 50  0000 C CNN
 	1    4900 3350
@@
 F 0 "R5" V 5380 3550 50  0000 C CNN
 F 1 "22" V 5300 3550 50  0000 C CNN
-F 2 "" V 5230 3550 50  0001 C CNN
+F 2 "Resistors_SMD:R_0402" V 5230 3550 50  0001 C CNN
 F 3 "" H 5300 3550 50  0000 C CNN
 	1    5300 3550
@@
 F 0 "R3" V 4980 3750 50  0000 C CNN
 F 1 "22" V 4900 3750 50  0000 C CNN
-F 2 "" V 4830 3750 50  0001 C CNN
+F 2 "Resistors_SMD:R_0402" V 4830 3750 50  0001 C CNN
 F 3 "" H 4900 3750 50  0000 C CNN
 	1    4900 3750
@@
 	3100 6050 3100 6000
 $Comp
-L LED D1
+L LED-RESCUE-interface D1
 U 1 1 59C78A89
 P 3100 5800
+AR Path="/59C78A89" Ref="D1"  Part="1"
+AR Path="/59C404DC/59C78A89" Ref="D1"  Part="1"
 F 0 "D1" H 3100 5900 50  0000 C CNN
 F 1 "ACTIVITY" H 3100 5700 50  0000 C CNN
@@
 F 0 "R1" V 3180 5450 50  0000 C CNN
 F 1 "330" V 3100 5450 50  0000 C CNN
-F 2 "" V 3030 5450 50  0001 C CNN
+F 2 "Resistors_SMD:R_0402" V 3030 5450 50  0001 C CNN
 F 3 "" H 3100 5450 50  0000 C CNN
 	1    3100 5450
@@
 F 0 "Q1" H 3200 6325 50  0000 L CNN
 F 1 "MMBF170" H 3200 6250 50  0000 L CNN
-F 2 "TO_SOT_Packages_SMD:SOT-23" H 3200 6175 50  0000 L CIN
+F 2 "TO_SOT_Packages_SMD:SOT-323_SC-70" H 3200 6175 50  0000 L CIN
 F 3 "" H 3000 6250 50  0000 L CNN
 	1    3000 6250
@@
 F 0 "R6" V 6130 2500 50  0000 C CNN
 F 1 "10K" V 6050 2500 50  0000 C CNN
-F 2 "" V 5980 2500 50  0001 C CNN
+F 2 "Resistors_SMD:R_0402" V 5980 2500 50  0001 C CNN
 F 3 "" H 6050 2500 50  0000 C CNN
 	1    6050 2500
@@
 F 0 "W5" H 5600 3020 50  0000 C CNN
 F 1 "CD" H 5600 2950 50  0000 C CNN
-F 2 "" H 5800 2750 50  0001 C CNN
+F 2 "Measurement_Points:Test_Point" H 5800 2750 50  0001 C CNN
 F 3 "" H 5800 2750 50  0000 C CNN
 	1    5600 2750

Commit message: Start of layout
Parts:
- Q1: footprint TO_SOT_Packages_SMD:SOT-323_SC-70 -> TO_SOT_Packages_SMD:SC-70
- SD1: footprint (none) -> SeeedOPL-Connector-2016:MICRO-SD9+4P-SMD-16.1X14.5X1.85MM
Changed lines of the file:
@@
 $EndDescr
 $Comp
-L GND #PWR01
+L GND #PWR5
 U 1 1 59C40584
 P 6600 4750
-F 0 "#PWR01" H 6600 4500 50  0001 C CNN
+F 0 "#PWR5" H 6600 4500 50  0001 C CNN
 F 1 "GND" H 6600 4600 50  0000 C CNN
 F 2 "" H 6600 4750 50  0000 C CNN
@@
 	6600 2000 6600 3450
 $Comp
-L +3.3V #PWR02
+L +3.3V #PWR4
 U 1 1 59C4084E
 P 6600 2000
-F 0 "#PWR02" H 6600 1850 50  0001 C CNN
+F 0 "#PWR4" H 6600 1850 50  0001 C CNN
 F 1 "+3.3V" H 6600 2140 50  0000 C CNN
 F 2 "" H 6600 2000 50  0000 C CNN
@@
 	7350 2200 7350 2400
 $Comp
-L GND #PWR03
+L GND #PWR6
 U 1 1 59C408FB
 P 7350 2400
-F 0 "#PWR03" H 7350 2150 50  0001 C CNN
+F 0 "#PWR6" H 7350 2150 50  0001 C CNN
 F 1 "GND" H 7350 2250 50  0000 C CNN
 F 2 "" H 7350 2400 50  0000 C CNN
@@
 SD_SPI_CS
 $Comp
-L GND #PWR04
+L GND #PWR2
 U 1 1 59C789EB
 P 3100 6600
-F 0 "#PWR04" H 3100 6350 50  0001 C CNN
+F 0 "#PWR2" H 3100 6350 50  0001 C CNN
 F 1 "GND" H 3100 6450 50  0000 C CNN
 F 2 "" H 3100 6600 50  0000 C CNN
@@
 $EndComp
 $Comp
-L +3.3V #PWR05
+L +3.3V #PWR1
 U 1 1 59C78BD3
 P 3100 5300
-F 0 "#PWR05" H 3100 5150 50  0001 C CNN
+F 0 "#PWR1" H 3100 5150 50  0001 C CNN
 F 1 "+3.3V" H 3100 5440 50  0000 C CNN
 F 2 "" H 3100 5300 50  0000 C CNN
@@
 F 0 "Q1" H 3200 6325 50  0000 L CNN
 F 1 "MMBF170" H 3200 6250 50  0000 L CNN
-F 2 "TO_SOT_Packages_SMD:SOT-323_SC-70" H 3200 6175 50  0000 L CIN
+F 2 "TO_SOT_Packages_SMD:SC-70" H 3200 6175 50  0000 L CIN
 F 3 "" H 3000 6250 50  0000 L CNN
 	1    3000 6250
@@
 F 0 "SD1" H 7050 4050 45  0000 L BNN
 F 1 "MICRO_SD" H 7400 3000 45  0000 L BNN
-F 2 "" H 7600 3550 79  0001 C CNN
+F 2 "SeeedOPL-Connector-2016:MICRO-SD9+4P-SMD-16.1X14.5X1.85MM" H 7600 3550 79  0001 C CNN
 F 3 "" H 7600 3550 79  0000 C CNN
 F 4 "ST-TF-003A" H 7630 3700 20  0001 C CNN "MPN"
@@
 Connection ~ 8000 4350
 $Comp
-L GND #PWR06
+L GND #PWR7
 U 1 1 59C9C2DA
 P 8400 4750
-F 0 "#PWR06" H 8400 4500 50  0001 C CNN
+F 0 "#PWR7" H 8400 4500 50  0001 C CNN
 F 1 "GND" H 8400 4600 50  0000 C CNN
 F 2 "" H 8400 4750 50  0000 C CNN
@@
 	1    0    0    -1
 $EndComp
-Wire Wire Line
-	6900 3650 6600 3650
-Wire Wire Line
-	6600 3650 6600 4750
 Wire Wire Line
 	6600 3450 6900 3450
@@
 	6050 2350 6050 2000
 $Comp
-L +3.3V #PWR07
+L +3.3V #PWR3
 U 1 1 59C9CAF7
 P 6050 2000
-F 0 "#PWR07" H 6050 1850 50  0001 C CNN
+F 0 "#PWR3" H 6050 1850 50  0001 C CNN
 F 1 "+3.3V" H 6050 2140 50  0000 C CNN
 F 2 "" H 6050 2000 50  0000 C CNN
@@
 	5600 2900 6050 2900
 Connection ~ 6050 2900
+Wire Wire Line
+	6900 3650 6600 3650
+Wire Wire Line
+	6600 3650 6600 4750
 $EndSCHEMATC
