File: interface/pcb/temp.sch (KiCad schematic (older format))
At the start: 10 parts, among them P3 TEMP/I2C, U3 LM75

Commit message: Partial BOM
Parts:
- W6, W7: footprint (none) -> Measurement_Points:Test_Point
Changed lines of the file:
@@
 EESchema Schematic File Version 2
+LIBS:interface-rescue
 LIBS:power
 LIBS:device
@@
 LIBS:tpd4s012
 LIBS:ap1509
-LIBS:device_big
 LIBS:SeeedOPL-Resistor-2016
 LIBS:SeeedOPL-Connector-2016
 LIBS:SeeedOPL-Inductor-2016
 LIBS:SeeedOPL-Display-2016
+LIBS:nhd-c0220biz
 LIBS:interface-cache
 EELAYER 25 0
@@
 	5450 4350 5450 4650
 $Comp
-L GND #PWR045
+L GND #PWR08
 U 1 1 59C73C46
 P 6600 4650
-F 0 "#PWR045" H 6600 4400 50  0001 C CNN
+F 0 "#PWR08" H 6600 4400 50  0001 C CNN
 F 1 "GND" H 6600 4500 50  0000 C CNN
 F 2 "" H 6600 4650 50  0000 C CNN
@@
 $EndComp
 $Comp
-L GND #PWR046
+L GND #PWR09
 U 1 1 59C73C6A
 P 5450 4650
-F 0 "#PWR046" H 5450 4400 50  0001 C CNN
+F 0 "#PWR09" H 5450 4400 50  0001 C CNN
 F 1 "GND" H 5450 4500 50  0000 C CNN
 F 2 "" H 5450 4650 50  0000 C CNN
@@
 $EndComp
 $Comp
-L +3.3V #PWR047
+L +3.3V #PWR010
 U 1 1 59C73C83
 P 6600 2100
-F 0 "#PWR047" H 6600 1950 50  0001 C CNN
+F 0 "#PWR010" H 6600 1950 50  0001 C CNN
 F 1 "+3.3V" H 6600 2240 50  0000 C CNN
 F 2 "" H 6600 2100 50  0000 C CNN
@@
 $EndComp
 $Comp
-L +3.3V #PWR048
+L +3.3V #PWR011
 U 1 1 59C73CA3
 P 7650 2100
-F 0 "#PWR048" H 7650 1950 50  0001 C CNN
+F 0 "#PWR011" H 7650 1950 50  0001 C CNN
 F 1 "+3.3V" H 7650 2240 50  0000 C CNN
 F 2 "" H 7650 2100 50  0000 C CNN
@@
 	5450 2750 5450 2900
 $Comp
-L GND #PWR049
+L GND #PWR012
 U 1 1 59C73F8F
 P 5450 2900
-F 0 "#PWR049" H 5450 2650 50  0001 C CNN
+F 0 "#PWR012" H 5450 2650 50  0001 C CNN
 F 1 "GND" H 5450 2750 50  0000 C CNN
 F 2 "" H 5450 2900 50  0000 C CNN
@@
 F 0 "W6" H 4500 2870 50  0000 C CNN
 F 1 "SCL" H 4500 2800 50  0000 C CNN
-F 2 "" H 4700 2600 50  0001 C CNN
+F 2 "Measurement_Points:Test_Point" H 4700 2600 50  0001 C CNN
 F 3 "" H 4700 2600 50  0000 C CNN
 	1    4500 2600
@@
 F 0 "W7" H 4600 3120 50  0000 C CNN
 F 1 "SDA" H 4600 3050 50  0000 C CNN
-F 2 "" H 4800 2850 50  0001 C CNN
+F 2 "Measurement_Points:Test_Point" H 4800 2850 50  0001 C CNN
 F 3 "" H 4800 2850 50  0000 C CNN
 	1    4600 2850
@@
 	3200 5300 3200 5450
 $Comp
-L GND #PWR050
+L GND #PWR013
 U 1 1 59C86C04
 P 3200 5450
-F 0 "#PWR050" H 3200 5200 50  0001 C CNN
+F 0 "#PWR013" H 3200 5200 50  0001 C CNN
 F 1 "GND" H 3200 5300 50  0000 C CNN
 F 2 "" H 3200 5450 50  0000 C CNN
@@
 $EndComp
 $Comp
-L +3.3V #PWR051
+L +3.3V #PWR014
 U 1 1 59C86C2D
 P 3200 4550
-F 0 "#PWR051" H 3200 4400 50  0001 C CNN
+F 0 "#PWR014" H 3200 4400 50  0001 C CNN
 F 1 "+3.3V" H 3200 4690 50  0000 C CNN
 F 2 "" H 3200 4550 50  0000 C CNN
@@
 $EndComp
 $Comp
-L GND #PWR052
+L GND #PWR015
 U 1 1 59C86CDF
 P 2250 4900
-F 0 "#PWR052" H 2250 4650 50  0001 C CNN
+F 0 "#PWR015" H 2250 4650 50  0001 C CNN
 F 1 "GND" H 2250 4750 50  0000 C CNN
 F 2 "" H 2250 4900 50  0000 C CNN

Commit message: Start of layout
Parts:
- P3: footprint (none) -> Sockets_MOLEX_KK-System:Socket_MOLEX-KK-RM2-54mm_Lock_4pin_straight
- R24, R25, R26, R27: footprint (none) -> Resistors_SMD:R_0402
- U3: footprint (none) -> Housings_SOIC:SOIC-8_3.9x4.9mm_Pitch1.27mm
Changed lines of the file:
@@
 F 0 "U3" H 6600 3600 59  0000 C CNN
 F 1 "LM75" H 6600 3700 59  0000 C CNN
-F 2 "" H 6600 3650 59  0001 C CNN
+F 2 "Housings_SOIC:SOIC-8_3.9x4.9mm_Pitch1.27mm" H 6600 3650 59  0001 C CNN
 F 3 "" H 6600 3650 59  0000 C CNN
 	1    6600 3650
@@
 F 0 "R26" V 6680 2400 50  0000 C CNN
 F 1 "0" V 6600 2400 50  0000 C CNN
-F 2 "" V 6530 2400 50  0001 C CNN
+F 2 "Resistors_SMD:R_0402" V 6530 2400 50  0001 C CNN
 F 3 "" H 6600 2400 50  0000 C CNN
 	1    6600 2400
@@
 F 0 "R24" V 5080 3450 50  0000 C CNN
 F 1 "22" V 5000 3450 50  0000 C CNN
-F 2 "" V 4930 3450 50  0001 C CNN
+F 2 "Resistors_SMD:R_0402" V 4930 3450 50  0001 C CNN
 F 3 "" H 5000 3450 50  0000 C CNN
 	1    5000 3450
@@
 F 0 "R25" V 5530 4200 50  0000 C CNN
 F 1 "0" V 5450 4200 50  0000 C CNN
-F 2 "" V 5380 4200 50  0001 C CNN
+F 2 "Resistors_SMD:R_0402" V 5380 4200 50  0001 C CNN
 F 3 "" H 5450 4200 50  0000 C CNN
 	1    5450 4200
@@
 F 0 "R27" V 7730 2400 50  0000 C CNN
 F 1 "56K" V 7650 2400 50  0000 C CNN
-F 2 "" V 7580 2400 50  0001 C CNN
+F 2 "Resistors_SMD:R_0402" V 7580 2400 50  0001 C CNN
 F 3 "" H 7650 2400 50  0000 C CNN
 	1    7650 2400
@@
 	5450 4350 5450 4650
 $Comp
-L GND #PWR08
+L GND #PWR14
 U 1 1 59C73C46
 P 6600 4650
-F 0 "#PWR08" H 6600 4400 50  0001 C CNN
+F 0 "#PWR14" H 6600 4400 50  0001 C CNN
 F 1 "GND" H 6600 4500 50  0000 C CNN
 F 2 "" H 6600 4650 50  0000 C CNN
@@
 $EndComp
 $Comp
-L GND #PWR09
+L GND #PWR12
 U 1 1 59C73C6A
 P 5450 4650
-F 0 "#PWR09" H 5450 4400 50  0001 C CNN
+F 0 "#PWR12" H 5450 4400 50  0001 C CNN
 F 1 "GND" H 5450 4500 50  0000 C CNN
 F 2 "" H 5450 4650 50  0000 C CNN
@@
 $EndComp
 $Comp
-L +3.3V #PWR010
+L +3.3V #PWR13
 U 1 1 59C73C83
 P 6600 2100
-F 0 "#PWR010" H 6600 1950 50  0001 C CNN
+F 0 "#PWR13" H 6600 1950 50  0001 C CNN
 F 1 "+3.3V" H 6600 2240 50  0000 C CNN
 F 2 "" H 6600 2100 50  0000 C CNN
@@
 $EndComp
 $Comp
-L +3.3V #PWR011
+L +3.3V #PWR15
 U 1 1 59C73CA3
 P 7650 2100
-F 0 "#PWR011" H 7650 1950 50  0001 C CNN
+F 0 "#PWR15" H 7650 1950 50  0001 C CNN
 F 1 "+3.3V" H 7650 2240 50  0000 C CNN
 F 2 "" H 7650 2100 50  0000 C CNN
@@
 	5450 2750 5450 2900
 $Comp
-L GND #PWR012
+L GND #PWR11
 U 1 1 59C73F8F
 P 5450 2900
-F 0 "#PWR012" H 5450 2650 50  0001 C CNN
+F 0 "#PWR11" H 5450 2650 50  0001 C CNN
 F 1 "GND" H 5450 2750 50  0000 C CNN
 F 2 "" H 5450 2900 50  0000 C CNN
@@
 F 0 "P3" H 2850 5400 50  0000 C CNN
 F 1 "TEMP/I2C" V 2950 5150 50  0000 C CNN
-F 2 "" H 2850 5150 50  0001 C CNN
+F 2 "Sockets_MOLEX_KK-System:Socket_MOLEX-KK-RM2-54mm_Lock_4pin_straight" H 2850 5150 50  0001 C CNN
 F 3 "" H 2850 5150 50  0000 C CNN
 	1    2850 5150
@@
 	3200 5300 3200 5450
 $Comp
-L GND #PWR013
+L GND #PWR10
 U 1 1 59C86C04
 P 3200 5450
-F 0 "#PWR013" H 3200 5200 50  0001 C CNN
+F 0 "#PWR10" H 3200 5200 50  0001 C CNN
 F 1 "GND" H 3200 5300 50  0000 C CNN
 F 2 "" H 3200 5450 50  0000 C CNN
@@
 $EndComp
 $Comp
-L +3.3V #PWR014
+L +3.3V #PWR9
 U 1 1 59C86C2D
 P 3200 4550
-F 0 "#PWR014" H 3200 4400 50  0001 C CNN
+F 0 "#PWR9" H 3200 4400 50  0001 C CNN
 F 1 "+3.3V" H 3200 4690 50  0000 C CNN
 F 2 "" H 3200 4550 50  0000 C CNN
@@
 $EndComp
 $Comp
-L GND #PWR015
+L GND #PWR8
 U 1 1 59C86CDF
 P 2250 4900
-F 0 "#PWR015" H 2250 4650 50  0001 C CNN
+F 0 "#PWR8" H 2250 4650 50  0001 C CNN
 F 1 "GND" H 2250 4750 50  0000 C CNN
 F 2 "" H 2250 4900 50  0000 C CNN
