File: interface/pcb/wiegand.sch (KiCad schematic (older format))
At the start: 20 parts, among them P4 CARD READER, Q3 MMBF170, Q4 MMBF170, Q5 MMBF170, Q6 MMBF170

Commit message: Partial BOM
Parts:
- W10, W11, W8, W9: footprint (none) -> Measurement_Points:Test_Point
Changed lines of the file:
@@
 EESchema Schematic File Version 2
+LIBS:interface-rescue
 LIBS:power
 LIBS:device
@@
 LIBS:tpd4s012
 LIBS:ap1509
-LIBS:device_big
 LIBS:SeeedOPL-Resistor-2016
 LIBS:SeeedOPL-Connector-2016
 LIBS:SeeedOPL-Inductor-2016
 LIBS:SeeedOPL-Display-2016
+LIBS:nhd-c0220biz
 LIBS:interface-cache
 EELAYER 25 0
@@
 $EndDescr
 $Comp
-L +12V #PWR053
+L +12V #PWR016
 U 1 1 59C747E2
 P 7000 2250
-F 0 "#PWR053" H 7000 2100 50  0001 C CNN
+F 0 "#PWR016" H 7000 2100 50  0001 C CNN
 F 1 "+12V" H 7000 2390 50  0000 C CNN
 F 2 "" H 7000 2250 50  0000 C CNN
@@
 	7000 4350 7000 5250
 $Comp
-L GND #PWR054
+L GND #PWR017
 U 1 1 59C74861
 P 7000 5250
-F 0 "#PWR054" H 7000 5000 50  0001 C CNN
+F 0 "#PWR017" H 7000 5000 50  0001 C CNN
 F 1 "GND" H 7000 5100 50  0000 C CNN
 F 2 "" H 7000 5250 50  0000 C CNN
@@
 	7950 3150 7950 3250
 $Comp
-L GND #PWR055
+L GND #PWR018
 U 1 1 59C7495D
 P 7550 3250
-F 0 "#PWR055" H 7550 3000 50  0001 C CNN
+F 0 "#PWR018" H 7550 3000 50  0001 C CNN
 F 1 "GND" H 7550 3100 50  0000 C CNN
 F 2 "" H 7550 3250 50  0000 C CNN
@@
 $EndComp
 $Comp
-L GND #PWR056
+L GND #PWR019
 U 1 1 59C74971
 P 7950 3250
-F 0 "#PWR056" H 7950 3000 50  0001 C CNN
+F 0 "#PWR019" H 7950 3000 50  0001 C CNN
 F 1 "GND" H 7950 3100 50  0000 C CNN
 F 2 "" H 7950 3250 50  0000 C CNN
@@
 	3600 4150 3600 4450
 $Comp
-L GND #PWR057
+L GND #PWR020
 U 1 1 59C74E49
 P 5650 5250
-F 0 "#PWR057" H 5650 5000 50  0001 C CNN
+F 0 "#PWR020" H 5650 5000 50  0001 C CNN
 F 1 "GND" H 5650 5100 50  0000 C CNN
 F 2 "" H 5650 5250 50  0000 C CNN
@@
 $EndComp
 $Comp
-L GND #PWR058
+L GND #PWR021
 U 1 1 59C74E66
 P 3600 5250
-F 0 "#PWR058" H 3600 5000 50  0001 C CNN
+F 0 "#PWR021" H 3600 5000 50  0001 C CNN
 F 1 "GND" H 3600 5100 50  0000 C CNN
 F 2 "" H 3600 5250 50  0000 C CNN
@@
 $EndComp
 $Comp
-L +3.3V #PWR059
+L +3.3V #PWR022
 U 1 1 59C75008
 P 5650 2250
-F 0 "#PWR059" H 5650 2100 50  0001 C CNN
+F 0 "#PWR022" H 5650 2100 50  0001 C CNN
 F 1 "+3.3V" H 5650 2390 50  0000 C CNN
 F 2 "" H 5650 2250 50  0000 C CNN
@@
 $EndComp
 $Comp
-L +3.3V #PWR060
+L +3.3V #PWR023
 U 1 1 59C75032
 P 5850 2250
-F 0 "#PWR060" H 5850 2100 50  0001 C CNN
+F 0 "#PWR023" H 5850 2100 50  0001 C CNN
 F 1 "+3.3V" H 5850 2390 50  0000 C CNN
 F 2 "" H 5850 2250 50  0000 C CNN
@@
 Connection ~ 5300 4700
 $Comp
-L GND #PWR061
+L GND #PWR024
 U 1 1 59C7554B
 P 4950 3100
-F 0 "#PWR061" H 4950 2850 50  0001 C CNN
+F 0 "#PWR024" H 4950 2850 50  0001 C CNN
 F 1 "GND" H 4950 2950 50  0000 C CNN
 F 2 "" H 4950 3100 50  0000 C CNN
@@
 $EndComp
 $Comp
-L +3.3V #PWR062
+L +3.3V #PWR025
 U 1 1 59C755C3
 P 4950 2250
-F 0 "#PWR062" H 4950 2100 50  0001 C CNN
+F 0 "#PWR025" H 4950 2100 50  0001 C CNN
 F 1 "+3.3V" H 4950 2390 50  0000 C CNN
 F 2 "" H 4950 2250 50  0000 C CNN
@@
 $EndComp
 $Comp
-L +3.3V #PWR063
+L +3.3V #PWR026
 U 1 1 59C75793
 P 4450 2250
-F 0 "#PWR063" H 4450 2100 50  0001 C CNN
+F 0 "#PWR026" H 4450 2100 50  0001 C CNN
 F 1 "+3.3V" H 4450 2390 50  0000 C CNN
 F 2 "" H 4450 2250 50  0000 C CNN
@@
 Connection ~ 4450 2800
 $Comp
-L GND #PWR064
+L GND #PWR027
 U 1 1 59C75966
 P 4450 3700
-F 0 "#PWR064" H 4450 3450 50  0001 C CNN
+F 0 "#PWR027" H 4450 3450 50  0001 C CNN
 F 1 "GND" H 4450 3550 50  0000 C CNN
 F 2 "" H 4450 3700 50  0000 C CNN
@@
 F 0 "W9" H 3500 2620 50  0000 C CNN
 F 1 "WG_1" H 3500 2550 50  0000 C CNN
-F 2 "" H 3700 2350 50  0001 C CNN
+F 2 "Measurement_Points:Test_Point" H 3700 2350 50  0001 C CNN
 F 3 "" H 3700 2350 50  0000 C CNN
 	1    3500 2350
@@
 F 0 "W10" H 3800 2620 50  0000 C CNN
 F 1 "WG_0" H 3800 2550 50  0000 C CNN
-F 2 "" H 4000 2350 50  0001 C CNN
+F 2 "Measurement_Points:Test_Point" H 4000 2350 50  0001 C CNN
 F 3 "" H 4000 2350 50  0000 C CNN
 	1    3800 2350
@@
 Connection ~ 7950 3950
 $Comp
-L GND #PWR065
+L GND #PWR028
 U 1 1 59C7686C
 P 7650 5250
-F 0 "#PWR065" H 7650 5000 50  0001 C CNN
+F 0 "#PWR028" H 7650 5000 50  0001 C CNN
 F 1 "GND" H 7650 5100 50  0000 C CNN
 F 2 "" H 7650 5250 50  0000 C CNN
@@
 $EndComp
 $Comp
-L GND #PWR066
+L GND #PWR029
 U 1 1 59C768B0
 P 7950 5250
-F 0 "#PWR066" H 7950 5000 50  0001 C CNN
+F 0 "#PWR029" H 7950 5000 50  0001 C CNN
 F 1 "GND" H 7950 5100 50  0000 C CNN
 F 2 "" H 7950 5250 50  0000 C CNN
@@
 F 0 "W8" H 3250 4820 50  0000 C CNN
 F 1 "LED" H 3250 4750 50  0000 C CNN
-F 2 "" H 3450 4550 50  0001 C CNN
+F 2 "Measurement_Points:Test_Point" H 3450 4550 50  0001 C CNN
 F 3 "" H 3450 4550 50  0000 C CNN
 	1    3250 4550
@@
 F 0 "W11" H 5300 4820 50  0000 C CNN
 F 1 "BUZZ" H 5300 4750 50  0000 C CNN
-F 2 "" H 5500 4550 50  0001 C CNN
+F 2 "Measurement_Points:Test_Point" H 5500 4550 50  0001 C CNN
 F 3 "" H 5500 4550 50  0000 C CNN
 	1    5300 4550

Commit message: Start of layout
Parts:
- C15: footprint Capacitors_Tantalum_SMD:TantalC_SizeB_EIA-3528_Reflow -> Capacitors_SMD:c_elec_6.3x5.3
- D2, D3: footprint (none) -> Diodes_SMD:SMA_Handsoldering
- P4: footprint (none) -> Sockets_MOLEX_KK-System:Socket_MOLEX-KK-RM2-54mm_Lock_6pin_straight
- Q3, Q4, Q5, Q6: footprint TO_SOT_Packages_SMD:SOT-23 -> TO_SOT_Packages_SMD:SC-70
- R28, R29, R30, R31, R32, R33, R34: footprint (none) -> Resistors_SMD:R_0402
Changed lines of the file:
@@
 $EndDescr
 $Comp
-L +12V #PWR016
+L +12V #PWR24
 U 1 1 59C747E2
 P 7000 2250
-F 0 "#PWR016" H 7000 2100 50  0001 C CNN
+F 0 "#PWR24" H 7000 2100 50  0001 C CNN
 F 1 "+12V" H 7000 2390 50  0000 C CNN
 F 2 "" H 7000 2250 50  0000 C CNN
@@
 F 0 "P4" H 8450 4450 50  0000 C CNN
 F 1 "CARD READER" V 8550 4100 50  0000 C CNN
-F 2 "" H 8450 4100 50  0001 C CNN
+F 2 "Sockets_MOLEX_KK-System:Socket_MOLEX-KK-RM2-54mm_Lock_6pin_straight" H 8450 4100 50  0001 C CNN
 F 3 "" H 8450 4100 50  0000 C CNN
 	1    8450 4100
@@
 	7000 4350 7000 5250
 $Comp
-L GND #PWR017
+L GND #PWR25
 U 1 1 59C74861
 P 7000 5250
-F 0 "#PWR017" H 7000 5000 50  0001 C CNN
+F 0 "#PWR25" H 7000 5000 50  0001 C CNN
 F 1 "GND" H 7000 5100 50  0000 C CNN
 F 2 "" H 7000 5250 50  0000 C CNN
@@
 F 0 "C15" H 7975 3100 50  0000 L CNN
 F 1 "10uF" H 7975 2900 50  0000 L CNN
-F 2 "Capacitors_Tantalum_SMD:TantalC_SizeB_EIA-3528_Reflow" H 7988 2850 50  0001 C CNN
+F 2 "Capacitors_SMD:c_elec_6.3x5.3" H 7988 2850 50  0001 C CNN
 F 3 "" H 7950 3000 50  0000 C CNN
 	1    7950 3000
@@
 	7950 3150 7950 3250
 $Comp
-L GND #PWR018
+L GND #PWR26
 U 1 1 59C7495D
 P 7550 3250
-F 0 "#PWR018" H 7550 3000 50  0001 C CNN
+F 0 "#PWR26" H 7550 3000 50  0001 C CNN
 F 1 "GND" H 7550 3100 50  0000 C CNN
 F 2 "" H 7550 3250 50  0000 C CNN
@@
 $EndComp
 $Comp
-L GND #PWR019
+L GND #PWR28
 U 1 1 59C74971
 P 7950 3250
-F 0 "#PWR019" H 7950 3000 50  0001 C CNN
+F 0 "#PWR28" H 7950 3000 50  0001 C CNN
 F 1 "GND" H 7950 3100 50  0000 C CNN
 F 2 "" H 7950 3250 50  0000 C CNN
@@
 F 0 "R34" V 7080 2500 50  0000 C CNN
 F 1 "0" V 7000 2500 50  0000 C CNN
-F 2 "" V 6930 2500 50  0001 C CNN
+F 2 "Resistors_SMD:R_0402" V 6930 2500 50  0001 C CNN
 F 3 "" H 7000 2500 50  0000 C CNN
 	1    7000 2500
@@
 	3600 4150 3600 4450
 $Comp
-L GND #PWR020
+L GND #PWR22
 U 1 1 59C74E49
 P 5650 5250
-F 0 "#PWR020" H 5650 5000 50  0001 C CNN
+F 0 "#PWR22" H 5650 5000 50  0001 C CNN
 F 1 "GND" H 5650 5100 50  0000 C CNN
 F 2 "" H 5650 5250 50  0000 C CNN
@@
 $EndComp
 $Comp
-L GND #PWR021
+L GND #PWR16
 U 1 1 59C74E66
 P 3600 5250
-F 0 "#PWR021" H 3600 5000 50  0001 C CNN
+F 0 "#PWR16" H 3600 5000 50  0001 C CNN
 F 1 "GND" H 3600 5100 50  0000 C CNN
 F 2 "" H 3600 5250 50  0000 C CNN
@@
 F 0 "R33" V 5930 2500 50  0000 C CNN
 F 1 "10K" V 5850 2500 50  0000 C CNN
-F 2 "" V 5780 2500 50  0001 C CNN
+F 2 "Resistors_SMD:R_0402" V 5780 2500 50  0001 C CNN
 F 3 "" H 5850 2500 50  0000 C CNN
 	1    5850 2500
@@
 F 0 "R32" V 5730 2500 50  0000 C CNN
 F 1 "10K" V 5650 2500 50  0000 C CNN
-F 2 "" V 5580 2500 50  0001 C CNN
+F 2 "Resistors_SMD:R_0402" V 5580 2500 50  0001 C CNN
 F 3 "" H 5650 2500 50  0000 C CNN
 	1    5650 2500
@@
 $EndComp
 $Comp
-L +3.3V #PWR022
+L +3.3V #PWR21
 U 1 1 59C75008
 P 5650 2250
-F 0 "#PWR022" H 5650 2100 50  0001 C CNN
+F 0 "#PWR21" H 5650 2100 50  0001 C CNN
 F 1 "+3.3V" H 5650 2390 50  0000 C CNN
 F 2 "" H 5650 2250 50  0000 C CNN
@@
 $EndComp
 $Comp
-L +3.3V #PWR023
+L +3.3V #PWR23
 U 1 1 59C75032
 P 5850 2250
-F 0 "#PWR023" H 5850 2100 50  0001 C CNN
+F 0 "#PWR23" H 5850 2100 50  0001 C CNN
 F 1 "+3.3V" H 5850 2390 50  0000 C CNN
 F 2 "" H 5850 2250 50  0000 C CNN
@@
 F 0 "R28" V 3330 5000 50  0000 C CNN
 F 1 "100K" V 3250 5000 50  0000 C CNN
-F 2 "" V 3180 5000 50  0001 C CNN
+F 2 "Resistors_SMD:R_0402" V 3180 5000 50  0001 C CNN
 F 3 "" H 3250 5000 50  0000 C CNN
 	1    3250 5000
@@
 F 0 "R31" V 5380 5000 50  0000 C CNN
 F 1 "100K" V 5300 5000 50  0000 C CNN
-F 2 "" V 5230 5000 50  0001 C CNN
+F 2 "Resistors_SMD:R_0402" V 5230 5000 50  0001 C CNN
 F 3 "" H 5300 5000 50  0000 C CNN
 	1    5300 5000
@@
 Connection ~ 5300 4700
 $Comp
-L GND #PWR024
+L GND #PWR20
 U 1 1 59C7554B
 P 4950 3100
-F 0 "#PWR024" H 4950 2850 50  0001 C CNN
+F 0 "#PWR20" H 4950 2850 50  0001 C CNN
 F 1 "GND" H 4950 2950 50  0000 C CNN
 F 2 "" H 4950 3100 50  0000 C CNN
@@
 F 0 "R30" V 5030 2500 50  0000 C CNN
 F 1 "10K" V 4950 2500 50  0000 C CNN
-F 2 "" V 4880 2500 50  0001 C CNN
+F 2 "Resistors_SMD:R_0402" V 4880 2500 50  0001 C CNN
 F 3 "" H 4950 2500 50  0000 C CNN
 	1    4950 2500
@@
 $EndComp
 $Comp
-L +3.3V #PWR025
+L +3.3V #PWR19
 U 1 1 59C755C3
 P 4950 2250
-F 0 "#PWR025" H 4950 2100 50  0001 C CNN
+F 0 "#PWR19" H 4950 2100 50  0001 C CNN
 F 1 "+3.3V" H 4950 2390 50  0000 C CNN
 F 2 "" H 4950 2250 50  0000 C CNN
@@
 F 0 "R29" V 4530 2500 50  0000 C CNN
 F 1 "10K" V 4450 2500 50  0000 C CNN
-F 2 "" V 4380 2500 50  0001 C CNN
+F 2 "Resistors_SMD:R_0402" V 4380 2500 50  0001 C CNN
 F 3 "" H 4450 2500 50  0000 C CNN
 	1    4450 2500
@@
 $EndComp
 $Comp
-L +3.3V #PWR026
+L +3.3V #PWR17
 U 1 1 59C75793
 P 4450 2250
-F 0 "#PWR026" H 4450 2100 50  0001 C CNN
+F 0 "#PWR17" H 4450 2100 50  0001 C CNN
 F 1 "+3.3V" H 4450 2390 50  0000 C CNN
 F 2 "" H 4450 2250 50  0000 C CNN
@@
 Connection ~ 4450 2800
 $Comp
-L GND #PWR027
+L GND #PWR18
 U 1 1 59C75966
 P 4450 3700
-F 0 "#PWR027" H 4450 3450 50  0001 C CNN
+F 0 "#PWR18" H 4450 3450 50  0001 C CNN
 F 1 "GND" H 4450 3550 50  0000 C CNN
 F 2 "" H 4450 3700 50  0000 C CNN
@@
 F 0 "D2" H 7450 4850 50  0000 C CNN
 F 1 "TVS" H 7650 4700 50  0000 C CNN
-F 2 "" H 7650 4800 50  0001 C CNN
+F 2 "Diodes_SMD:SMA_Handsoldering" H 7650 4800 50  0001 C CNN
 F 3 "" H 7650 4800 50  0000 C CNN
 	1    7650 4800
@@
 F 0 "D3" H 7750 4850 50  0000 C CNN
 F 1 "TVS" H 7950 4700 50  0000 C CNN
-F 2 "" H 7950 4800 50  0001 C CNN
+F 2 "Diodes_SMD:SMA_Handsoldering" H 7950 4800 50  0001 C CNN
 F 3 "" H 7950 4800 50  0000 C CNN
 	1    7950 4800
@@
 Connection ~ 7950 3950
 $Comp
-L GND #PWR028
+L GND #PWR27
 U 1 1 59C7686C
 P 7650 5250
-F 0 "#PWR028" H 7650 5000 50  0001 C CNN
+F 0 "#PWR27" H 7650 5000 50  0001 C CNN
 F 1 "GND" H 7650 5100 50  0000 C CNN
 F 2 "" H 7650 5250 50  0000 C CNN
@@
 $EndComp
 $Comp
-L GND #PWR029
+L GND #PWR29
 U 1 1 59C768B0
 P 7950 5250
-F 0 "#PWR029" H 7950 5000 50  0001 C CNN
+F 0 "#PWR29" H 7950 5000 50  0001 C CNN
 F 1 "GND" H 7950 5100 50  0000 C CNN
 F 2 "" H 7950 5250 50  0000 C CNN
@@
 F 0 "Q3" H 3700 4725 50  0000 L CNN
 F 1 "MMBF170" H 3700 4650 50  0000 L CNN
-F 2 "TO_SOT_Packages_SMD:SOT-23" H 3700 4575 50  0000 L CIN
+F 2 "TO_SOT_Packages_SMD:SC-70" H 3700 4575 50  0000 L CIN
 F 3 "" H 3500 4650 50  0000 L CNN
 	1    3500 4650
@@
 F 0 "Q6" H 5750 4725 50  0000 L CNN
 F 1 "MMBF170" H 5750 4650 50  0000 L CNN
-F 2 "TO_SOT_Packages_SMD:SOT-23" H 5750 4575 50  0000 L CIN
+F 2 "TO_SOT_Packages_SMD:SC-70" H 5750 4575 50  0000 L CIN
 F 3 "" H 5550 4650 50  0000 L CNN
 	1    5550 4650
@@
 F 0 "Q4" H 4750 3575 50  0000 L CNN
 F 1 "MMBF170" H 4750 3500 50  0000 L CNN
-F 2 "TO_SOT_Packages_SMD:SOT-23" H 4750 3425 50  0000 L CIN
+F 2 "TO_SOT_Packages_SMD:SC-70" H 4750 3425 50  0000 L CIN
 F 3 "" H 4550 3500 50  0000 L CNN
 	1    4550 3500
@@
 F 0 "Q5" H 5250 2975 50  0000 L CNN
 F 1 "MMBF170" H 5250 2900 50  0000 L CNN
-F 2 "TO_SOT_Packages_SMD:SOT-23" H 5250 2825 50  0000 L CIN
+F 2 "TO_SOT_Packages_SMD:SC-70" H 5250 2825 50  0000 L CIN
 F 3 "" H 5050 2900 50  0000 L CNN
 	1    5050 2900
